Commit message: Support for ros2 jazzy
Signed-off-by: Juancams <jc.manzanares.serrano@gmail.com>

File: kobuki_description/urdf/asus_xtion_pro_offset.urdf.xacro (robot description, xacro)
@@ -33,5 +33,5 @@
         <origin xyz="-0.01 0 0" rpy="${-M_PI/2} -${M_PI} ${-M_PI/2}"/>
         <geometry>
-          <mesh filename="package://kobuki_description/meshes/sensors/asus_xtion_pro_live.dae" scale="${M_SCALE} ${M_SCALE} ${M_SCALE}"/>
+          <mesh filename="file://$(find kobuki_description)/meshes/sensors/asus_xtion_pro_live.dae" scale="${M_SCALE} ${M_SCALE} ${M_SCALE}"/>
         </geometry>
       </visual>

File: kobuki_description/urdf/hexagons.urdf.xacro (robot description, xacro)
@@ -19,5 +19,5 @@
         <origin xyz="0 0 0" rpy="0 0 0"/>
         <geometry>
-          <mesh filename="package://kobuki_description/meshes/stacks/hexagons/pole_bottom.dae"/>
+          <mesh filename="file://$(find kobuki_description)/meshes/stacks/hexagons/pole_bottom.dae"/>
         </geometry>
       </visual>
@@ -47,5 +47,5 @@
         <origin xyz="0 0 0" rpy="0 ${M_PI} 0"/>
         <geometry>
-          <mesh filename="package://kobuki_description/meshes/stacks/hexagons/pole_middle.dae"/>
+          <mesh filename="file://$(find kobuki_description)/meshes/stacks/hexagons/pole_middle.dae"/>
         </geometry>
       </visual>
@@ -75,5 +75,5 @@
         <origin xyz=" 0 0 0" rpy="0 0 0"/>
         <geometry>
-          <mesh filename="package://kobuki_description/meshes/stacks/hexagons/pole_top.dae"/>
+          <mesh filename="file://$(find kobuki_description)/meshes/stacks/hexagons/pole_top.dae"/>
         </geometry>
       </visual>
@@ -103,5 +103,5 @@
         <origin xyz="0 0 -0.01" rpy="0 0 0"/>
         <geometry>
-          <mesh filename="package://kobuki_description/meshes/sensors/sensor_pole.dae" />
+          <mesh filename="file://$(find kobuki_description)/meshes/sensors/sensor_pole.dae" />
         </geometry>
       </visual>
@@ -142,5 +142,5 @@
         <origin xyz="0 0 0" rpy="0 0 0"/>
         <geometry>
-          <mesh filename="package://kobuki_description/meshes/stacks/hexagons/plate_bottom.dae"/>
+          <mesh filename="file://$(find kobuki_description)/meshes/stacks/hexagons/plate_bottom.dae"/>
         </geometry>
       </visual>
@@ -172,5 +172,5 @@
         <origin xyz="0 0 0" rpy="0 0 0"/>
         <geometry>
-          <mesh filename="package://kobuki_description/meshes/stacks/hexagons/plate_middle.dae"/>
+          <mesh filename="file://$(find kobuki_description)/meshes/stacks/hexagons/plate_middle.dae"/>
         </geometry>
       </visual>
@@ -204,5 +204,5 @@
         <origin xyz="0 0 0" rpy="0 0 0"/>
         <geometry>
-          <mesh filename="package://kobuki_description/meshes/stacks/hexagons/plate_top.dae"/>
+          <mesh filename="file://$(find kobuki_description)/meshes/stacks/hexagons/plate_top.dae"/>
         </geometry>
       </visual>

File: kobuki_description/urdf/kobuki.urdf.xacro (robot description, xacro)
@@ -6,8 +6,8 @@
       kobuki_description/launch/view_model.launch
  -->
-<robot name="kobuki" xmlns:xacro="http://ros.org/wiki/xacro">
+<robot name="kobuki" xmlns:xacro="http://ros.org/wiki/xacro" parmas= prefix>
   <xacro:include filename="$(find kobuki_description)/urdf/common_properties.urdf.xacro"/>
   <!-- Kobuki -->
-  <xacro:macro name="kobuki">
+  <xacro:macro name="$(prefix)_kobuki">
     <link name="base_footprint"/>
     <!--

File: kobuki_description/urdf/kobuki_gazebo.urdf.xacro (robot description, xacro)
@@ -29,5 +29,5 @@
         <geometry>
           <!-- new mesh -->
-          <mesh filename="package://kobuki_description/meshes/main_body.dae" />
+          <mesh filename="file://$(find kobuki_description)/meshes/main_body.dae" />
         </geometry>
         <origin xyz="0.001 0 0.05199" rpy="0 0 0"/>
@@ -64,5 +64,5 @@
       <visual>
         <geometry>
-          <mesh filename="package://kobuki_description/meshes/wheel.dae"/>
+          <mesh filename="file://$(find kobuki_description)/meshes/wheel.dae"/>
         </geometry>
         <origin xyz="0 0 0" rpy="0 0 0"/>
@@ -91,5 +91,5 @@
       <visual>
         <geometry>
-          <mesh filename="package://kobuki_description/meshes/wheel.dae"/>
+          <mesh filename="file://$(find kobuki_description)/meshes/wheel.dae"/>
         </geometry>
         <origin xyz="0 0 0" rpy="0 0 0"/>
@@ -208,22 +208,20 @@
     </link>
     <gazebo>
-      <plugin name="differential_drive_controller" filename="libgazebo_ros_diff_drive.so">
-        <update_rate>10</update_rate>
+      <plugin filename="gz-sim-diff-drive-system" name="gz::sim::systems::DiffDrive">
+        <!-- Remove <ros> tag. -->
+        <!-- wheels -->
         <left_joint>wheel_left_joint</left_joint>
         <right_joint>wheel_right_joint</right_joint>
-        <wheel_separation>0.230</wheel_separation>
-        <wheel_diameter>0.070</wheel_diameter>
-        <max_wheel_torque>1.0</max_wheel_torque>
-        <max_wheel_acceleration>1.0</max_wheel_acceleration>
-        <command_topic>cmd_vel</command_topic>
-        <!-- output -->
-        <publish_odom>true</publish_odom>
-        <publish_odom_tf>true</publish_odom_tf>
-        <publish_wheel_tf>true</publish_wheel_tf>
-        <odometry_topic>odom</odometry_topic>
-        <odometry_frame>odom</odometry_frame>
-        <robot_base_frame>base_link</robot_base_frame>
-	    </plugin>
-	  </gazebo>
+        <!-- kinematics -->
+        <wheel_separation>0.223087</wheel_separation>
+        <wheel_radius>0.035</wheel_radius> <!-- computed from <wheel_diameter> in the original plugin-->
+        <!-- limits -->
+        <max_linear_acceleration>1.0</max_linear_acceleration> <!-- computed from <max_linear_acceleration> in the original plugin-->
+        <topic>cmd_vel</topic> <!-- from <commant_topic> -->
+        <child_frame_id>base_footprint</child_frame_id> <!-- from <robot_base_frame> -->
+        <odom_publisher_frequency>30</odom_publisher_frequency> <!-- from <update_rate>-->
+        <tf_topic>/tf</tf_topic> <!-- Short topic name for tf output -->
+      </plugin>
+    </gazebo>
      <gazebo reference="camera_link">
   <sensor name="camera" type="depth">
@@ -241,5 +239,5 @@
       </clip>
     </camera>
-    <plugin name="camera_controller" filename="libgazebo_ros_camera.so">
+    <!-- <plugin name="camera_controller" filename="libgazebo_ros_camera.so">
       <baseline>0.2</baseline>
       <alwaysOn>true</alwaysOn>
@@ -258,5 +256,5 @@
       <focalLength>0</focalLength>
       <hackBaseline>0</hackBaseline>
-    </plugin>
+    </plugin> -->
   </sensor>
 </gazebo>
@@ -269,5 +267,5 @@
 	<visual>
         <geometry>
-          <mesh filename="package://kobuki_description/meshes/sensors/rplidar.dae" scale="0.001 0.001 0.001" />
+          <mesh filename="file://$(find kobuki_description)/meshes/sensors/rplidar.dae" scale="0.001 0.001 0.001" />
         </geometry>
         <origin xyz="0 0 0.025" rpy="-1.5707 0 -1.5707"/>
@@ -306,5 +304,5 @@
         </noise>
       </ray>
-      <plugin filename="libgazebo_ros_ray_sensor.so" name="scan">
+      <!-- <plugin filename="libgazebo_ros_ray_sensor.so" name="scan">
         <ros>
           <remapping>~/out:=scan</remapping>
@@ -312,5 +310,5 @@
         <output_type>sensor_msgs/LaserScan</output_type>
         <frame_name>laser_link</frame_name>
-      </plugin>
+      </plugin> -->
     </sensor>
   </gazebo>

File: kobuki_description/urdf/sensors/asus_xtion_pro.urdf.xacro (robot description, xacro)
@@ -33,5 +33,5 @@
         <origin xyz="-0.015 0.0035 0.004" rpy="0 0 0"/>
         <geometry>
-          <mesh filename="package://kobuki_description/meshes/sensors/xtion_pro_camera.dae"/>
+          <mesh filename="file://$(find kobuki_description)/meshes/sensors/xtion_pro_camera.dae"/>
         </geometry>
       </visual>
@@ -74,5 +74,5 @@
         <origin xyz="0 0 0" rpy="${-M_PI/2} 0 0"/>
         <geometry>
-          <mesh filename="package://kobuki_description/meshes/sensors/xtion_pro_stack.dae"/>
+          <mesh filename="file://$(find kobuki_description)/meshes/sensors/xtion_pro_stack.dae"/>
         </geometry>
       </visual>

File: kobuki_description/urdf/stacks/circles.urdf.xacro (robot description, xacro)
@@ -18,5 +18,5 @@
         <origin xyz=" 0 0 0 " rpy="0 0 0" />
         <geometry>
-          <mesh filename="package://kobuki_description/meshes/stacks/circles/68-02403-125_Spacer.dae"/>
+          <mesh filename="file://$(find kobuki_description)/meshes/stacks/circles/68-02403-125_Spacer.dae"/>
         </geometry>
       </visual>
@@ -46,5 +46,5 @@
         <origin xyz=" 0 0 0 " rpy="0 0 0" />
         <geometry>
-          <mesh filename="package://kobuki_description/meshes/stacks/circles/68-04552-1000-RA_Turtlebot_M-F_Standoff.dae"/>
+          <mesh filename="file://$(find kobuki_description)/meshes/stacks/circles/68-04552-1000-RA_Turtlebot_M-F_Standoff.dae"/>
         </geometry>
       </visual>
@@ -74,5 +74,5 @@
         <origin xyz=" 0 0 0 " rpy="0 0 0" />
         <geometry>
-          <mesh filename="package://kobuki_description/meshes/stacks/circles/68-04552-2000-RA_Turtlebot_M-F_Standoff.dae"/>
+          <mesh filename="file://$(find kobuki_description)/meshes/stacks/circles/68-04552-2000-RA_Turtlebot_M-F_Standoff.dae"/>
         </geometry>
       </visual>
@@ -102,5 +102,5 @@
         <origin xyz=" 0 0 0 " rpy="0 0 0" />
         <geometry>
-          <mesh filename="package://kobuki_description/meshes/stacks/circles/68-02421-8000-RA_Turtlebot_F-F_Standoff.dae"/>
+          <mesh filename="file://$(find kobuki_description)/meshes/stacks/circles/68-02421-8000-RA_Turtlebot_F-F_Standoff.dae"/>
         </geometry>
       </visual>
@@ -130,5 +130,5 @@
         <origin xyz=" 0 0 0 " rpy="0 0 0" />
         <geometry>
-          <mesh filename="package://kobuki_description/meshes/stacks/circles/68-04556-RA_Kinect_Standoff_Assy.dae"/>
+          <mesh filename="file://$(find kobuki_description)/meshes/stacks/circles/68-04556-RA_Kinect_Standoff_Assy.dae"/>
         </geometry>
       </visual>
@@ -162,5 +162,5 @@
         <origin xyz=" 0 0 0 " rpy="0 0 0" />
         <geometry>
-          <mesh filename="package://kobuki_description/meshes/stacks/circles/plate_0_logo.dae"/>
+          <mesh filename="file://$(find kobuki_description)/meshes/stacks/circles/plate_0_logo.dae"/>
         </geometry>
       </visual>
@@ -192,5 +192,5 @@
         <origin xyz=" 0 0 0 " rpy="0 0 0" />
         <geometry>
-          <mesh filename="package://kobuki_description/meshes/stacks/circles/plate_1_logo.dae"/>
+          <mesh filename="file://$(find kobuki_description)/meshes/stacks/circles/plate_1_logo.dae"/>
         </geometry>
       </visual>
@@ -222,5 +222,5 @@
         <origin xyz=" 0 0 0 " rpy="0 0 0" />
         <geometry>
-          <mesh filename="package://kobuki_description/meshes/stacks/circles/plate_1_logo.dae"/>
+          <mesh filename="file://$(find kobuki_description)/meshes/stacks/circles/plate_1_logo.dae"/>
         </geometry>
       </visual>
@@ -254,5 +254,5 @@
         <origin xyz=" 0 0 0 " rpy="0 0 0" />
         <geometry>
-          <mesh filename="package://kobuki_description/meshes/stacks/circles/plate_2_logo.dae"/>
+          <mesh filename="file://$(find kobuki_description)/meshes/stacks/circles/plate_2_logo.dae"/>
         </geometry>
       </visual>
