Commit message: Added use_sim_time, new bridges & joint_states
Signed-off-by: Juancams <jc.manzanares.serrano@gmail.com>

File: kobuki_description/urdf/kobuki_gazebo.urdf.xacro (robot description, xacro)
@@ -15,4 +15,9 @@
         <odom_publisher_frequency>30</odom_publisher_frequency>
         <tf_topic>/tf</tf_topic>
+      </plugin>
+      <plugin filename="gz-sim-joint-state-publisher-system" name="gz::sim::systems::JointStatePublisher">
+        <topic>joint_states</topic>
+        <joint>wheel_left_joint</joint>
+        <joint>wheel_right_joint</joint>
       </plugin>
     </gazebo>

Commit message: laser fixed, rviz comprobations done

File: kobuki_description/urdf/kobuki_gazebo.urdf.xacro (robot description, xacro)
@@ -28,11 +28,11 @@
       <render_engine>ogre2</render_engine>
     </plugin>
-      <gazebo reference="laser_link">
-        <sensor name="kobuki_lidar" type="gpu_lidar">
+      <gazebo reference="$(arg namespace)/laser_link">
+        <sensor name="$(arg namespace)/kobuki_lidar" type="gpu_lidar">
             <always_on>true</always_on>
             <visualize>true</visualize>
             <update_rate>5</update_rate>
             <topic>$(arg namespace)/scan_raw</topic>
-            <gz_frame_id>laser_link</gz_frame_id>
+            <gz_frame_id>$(arg namespace)/laser_link</gz_frame_id>
             <lidar>
               <scan>

File: kobuki_description/urdf/sensors/r200.urdf.xacro (robot description, xacro)
@@ -88,5 +88,5 @@
           <box size="0.130 0.567 0.118"/>
         </geometry>
-      </collision>-->
+      </collision>
       <!-- This inertial field needs doesn't contain reliable data!! -->
      <inertial>
