Commit message: Add multirobot support
Signed-off-by: Francisco Martín Rico <fmrico@gmail.com>

File: kobuki_description/urdf/kobuki_base.urdf.xacro (robot description, xacro)
@@ -9,6 +9,6 @@
   <xacro:include filename="$(find kobuki_description)/urdf/common_properties.urdf.xacro"/>
   <!-- Kobuki -->
-  <xacro:macro name="kobuki_base">
-    <link name="base_footprint"/>
+  <xacro:macro name="kobuki_base" params = "namespace">
+    <link name="$(arg namespace)base_footprint"/>
     <!--
        Base link is set at the bottom of the base mould.
@@ -20,10 +20,10 @@
        to 0.352.
       -->
-    <joint name="base_joint" type="fixed">
+    <joint name="$(arg namespace)base_joint" type="fixed">
       <origin xyz="0 0 0.0102" rpy="0 0 0" />
-      <parent link="base_footprint"/>
-      <child link="base_link" />
-    </joint>
-    <link name="base_link">
+      <parent link="$(arg namespace)base_footprint"/>
+      <child link="$(arg namespace)base_link" />
+    </joint>
+    <link name="$(arg namespace)base_link">
       <visual>
         <geometry>
@@ -55,11 +55,11 @@
       </inertial>
     </link>
-    <joint name="wheel_left_joint" type="continuous">
-      <parent link="base_link"/>
-      <child link="wheel_left_link"/>
-      <origin xyz="0.00 ${0.23/2} 0.0250" rpy="${-M_PI/2} 0 0"/>
+    <joint name="$(arg namespace)wheel_left_joint" type="continuous">
+      <parent link="$(arg namespace)base_link"/>
+      <child link="$(arg namespace)wheel_left_link"/>
+      <origin xyz="0.00 ${0.25/2} 0.0250" rpy="${-M_PI/2} 0 0"/>
       <axis xyz="0 0 1"/>
     </joint>
-    <link name="wheel_left_link">
+    <link name="$(arg namespace)wheel_left_link">
       <visual>
         <geometry>
@@ -82,11 +82,11 @@
       </inertial>
     </link>
-    <joint name="wheel_right_joint" type="continuous">
-      <parent link="base_link"/>
-      <child link="wheel_right_link"/>
-      <origin xyz="0.00 -${0.23/2} 0.0250" rpy="${-M_PI/2} 0 0"/>
+    <joint name="$(arg namespace)wheel_right_joint" type="continuous">
+      <parent link="$(arg namespace)base_link"/>
+      <child link="$(arg namespace)wheel_right_link"/>
+      <origin xyz="0.00 -${0.25/2} 0.0250" rpy="${-M_PI/2} 0 0"/>
       <axis xyz="0 0 1"/>
     </joint>
-    <link name="wheel_right_link">
+    <link name="$(arg namespace)wheel_right_link">
       <visual>
         <geometry>
@@ -109,10 +109,10 @@
       </inertial>
     </link>
-    <joint name="caster_front_joint" type="fixed">
-      <parent link="base_link"/>
-      <child link="caster_front_link"/>
+    <joint name="$(arg namespace)caster_front_joint" type="fixed">
+      <parent link="$(arg namespace)base_link"/>
+      <child link="$(arg namespace)caster_front_link"/>
       <origin xyz="0.115 0.0 0.007" rpy="${-M_PI/2} 0 0"/>
     </joint>
-    <link name="caster_front_link">
+    <link name="$(arg namespace)caster_front_link">
       <collision>
         <geometry>
@@ -129,10 +129,10 @@
       </inertial>
     </link>
-    <joint name="caster_back_joint" type="fixed">
-      <parent link="base_link"/>
-      <child link="caster_back_link"/>
+    <joint name="$(arg namespace)caster_back_joint" type="fixed">
+      <parent link="$(arg namespace)base_link"/>
+      <child link="$(arg namespace)caster_back_link"/>
       <origin xyz="-0.135 0.0 0.009" rpy="${-M_PI/2} 0 0"/>
     </joint>
-    <link name="caster_back_link">
+    <link name="$(arg namespace)caster_back_link">
       <collision>
         <geometry>
@@ -150,11 +150,11 @@
     </link>
     <!-- Kobuki's sensors -->
-    <joint name="gyro_joint" type="fixed">
+    <joint name="$(arg namespace)gyro_joint" type="fixed">
       <axis xyz="0 1 0"/>
       <origin xyz="0.056 0.062 0.0202" rpy="0 0 0"/>
-      <parent link="base_link"/>
-      <child link="gyro_link"/>
-    </joint>
-    <link name="gyro_link">
+      <parent link="$(arg namespace)base_link"/>
+      <child link="$(arg namespace)gyro_link"/>
+    </joint>
+    <link name="$(arg namespace)gyro_link">
       <inertial>
         <mass value="0.001"/>
@@ -165,10 +165,10 @@
       </inertial>
     </link>
-    <joint name="cliff_sensor_left_joint" type="fixed">
+    <joint name="$(arg namespace)cliff_sensor_left_joint" type="fixed">
       <origin xyz="0.08734 0.13601 0.0214" rpy="0 ${M_PI/2} 0" />
-      <parent link="base_link"/>
-      <child link="cliff_sensor_left_link" />
-    </joint>
-    <link name="cliff_sensor_left_link">
+      <parent link="$(arg namespace)base_link"/>
+      <child link="$(arg namespace)cliff_sensor_left_link" />
+    </joint>
+    <link name="$(arg namespace)cliff_sensor_left_link">
       <inertial>
         <mass value="0.0001" />
@@ -179,10 +179,10 @@
       </inertial>
     </link>
-    <joint name="cliff_sensor_right_joint" type="fixed">
+    <joint name="$(arg namespace)cliff_sensor_right_joint" type="fixed">
       <origin xyz="0.085 -0.13601 0.0214" rpy="0 ${M_PI/2} 0" />
-      <parent link="base_link"/>
-      <child link="cliff_sensor_right_link" />
-    </joint>
-    <link name="cliff_sensor_right_link">
+      <parent link="$(arg namespace)base_link"/>
+      <child link="$(arg namespace)cliff_sensor_right_link" />
+    </joint>
+    <link name="$(arg namespace)cliff_sensor_right_link">
       <inertial>
         <mass value="0.0001" />
@@ -193,10 +193,10 @@
       </inertial>
     </link>
-    <joint name="cliff_sensor_front_joint" type="fixed">
+    <joint name="$(arg namespace)cliff_sensor_front_joint" type="fixed">
       <origin xyz="0.156 0.00 0.0214" rpy="0 ${M_PI/2} 0" />
-      <parent link="base_link"/>
-      <child link="cliff_sensor_front_link" />
-    </joint>
-    <link name="cliff_sensor_front_link">
+      <parent link="$(arg namespace)base_link"/>
+      <child link="$(arg namespace)cliff_sensor_front_link" />
+    </joint>
+    <link name="$(arg namespace)cliff_sensor_front_link">
       <inertial>
         <mass value="0.0001" />

File: kobuki_description/urdf/kobuki_gazebo.urdf.xacro (robot description, xacro)
@@ -1,23 +1,23 @@
 <?xml version="1.0" ?>
 <robot name="kobuki_gazebo" xmlns:xacro="http://ros.org/wiki/xacro">
-  <xacro:macro name="kobuki_gazebo" params="lidar camera">
+  <xacro:macro name="kobuki_gazebo" params="lidar camera namespace tf_namespace">
     <gazebo>
       <plugin filename="gz-sim-diff-drive-system" name="gz::sim::systems::DiffDrive">
-        <left_joint>wheel_left_joint</left_joint>
-        <right_joint>wheel_right_joint</right_joint>
+        <left_joint>$(arg namespace)wheel_left_joint</left_joint>
+        <right_joint>$(arg namespace)wheel_right_joint</right_joint>
         <wheel_separation>0.223087</wheel_separation>
         <wheel_radius>0.035</wheel_radius>
         <max_linear_acceleration>1.0</max_linear_acceleration>
-        <topic>cmd_vel</topic>
-        <odom_topic>odom</odom_topic>
-        <frame_id>odom</frame_id>
-        <child_frame_id>base_footprint</child_frame_id>
+        <topic>$(arg namespace)cmd_vel</topic>
+        <odom_topic>$(arg namespace)odom</odom_topic>
+        <frame_id>$(arg namespace)odom</frame_id>
+        <child_frame_id>$(arg namespace)base_footprint</child_frame_id>
         <odom_publisher_frequency>30</odom_publisher_frequency>
-        <tf_topic>/tf</tf_topic>
+        <tf_topic>$(arg tf_namespace)tf</tf_topic>
       </plugin>
       <plugin filename="gz-sim-joint-state-publisher-system" name="gz::sim::systems::JointStatePublisher">
-        <topic>joint_states</topic>
-        <joint>wheel_left_joint</joint>
-        <joint>wheel_right_joint</joint>
+        <topic>$(arg namespace)joint_states</topic>
+        <joint>$(arg namespace)wheel_left_joint</joint>
+        <joint>$(arg namespace)wheel_right_joint</joint>
       </plugin>
     </gazebo>
@@ -28,11 +28,11 @@
       <render_engine>ogre2</render_engine>
     </plugin>
-      <gazebo reference="laser_link">
-        <sensor name="kobuki_lidar" type="gpu_lidar">
+      <gazebo reference="$(arg namespace)laser_link">
+        <sensor name="$(arg namespace)kobuki_lidar" type="gpu_lidar">
             <always_on>true</always_on>
             <visualize>true</visualize>
             <update_rate>5</update_rate>
-            <topic>scan_raw</topic>
-            <gz_frame_id>laser_link</gz_frame_id>
+            <topic>$(arg namespace)scan_raw</topic>
+            <gz_frame_id>$(arg namespace)laser_link</gz_frame_id>
             <lidar>
               <scan>
@@ -59,10 +59,10 @@
     </xacro:if>
     <xacro:if value="$(arg camera)">
-      <gazebo reference="camera_rgb_frame">
-        <sensor type="rgbd_camera" name="kobuki_frame_sensor">
+      <gazebo reference="$(arg namespace)camera_rgb_frame">
+        <sensor type="rgbd_camera" name="$(arg namespace)kobuki_frame_sensor">
           <always_on>1</always_on>
           <update_rate>30.0</update_rate>
           <visualize>true</visualize>
-          <topic>rgbd_camera</topic>
+          <topic>$(arg namespace)rgbd_camera</topic>
           <camera>
             <horizontal_fov>${63.0*M_PI/180.0}</horizontal_fov>
@@ -83,5 +83,5 @@
               <p2>0.00000001</p2>
             </distortion>
-            <optical_frame_id>camera_rgb_optical_frame</optical_frame_id>
+            <optical_frame_id>$(arg namespace)camera_link</optical_frame_id>
           </camera>
         </sensor>
