Commit message: Reformat all xacros
Signed-off-by: Juancams <jc.manzanares.serrano@gmail.com>

File: kobuki_description/urdf/kobuki_gazebo.urdf.xacro (robot description, xacro)
@@ -1,316 +1,52 @@
 <?xml version="1.0" ?>
-<!--
-  This is not a standalone urdf for kobuki. It simply defines the 'kobuki' tag that can
-  be incorporated by other urdf files (e.g. turtlebot).
-  See kobuki_standalone.urdf.xacro for a standalone urdf to be tested with
-      kobuki_description/launch/view_model.launch
- -->
-<robot name="kobuki" xmlns:xacro="http://ros.org/wiki/xacro">
-  <xacro:include filename="$(find kobuki_description)/urdf/common_properties.urdf.xacro"/>
-  <!-- Kobuki -->
-  <xacro:macro name="kobuki">
-    <link name="base_footprint"/>
-    <!--
-       Base link is set at the bottom of the base mould.
-       This is done to be compatible with the way base link
-       was configured for turtlebot 1. Refer to
-       https://github.com/turtlebot/turtlebot/issues/40
-       To put the base link at the more oft used wheel
-       axis, set the z-distance from the base_footprint
-       to 0.352.
-      -->
-    <joint name="base_joint" type="fixed">
-      <origin xyz="0 0 0.0102" rpy="0 0 0" />
-      <parent link="base_footprint"/>
-      <child link="base_link" />
-    </joint>
-    <link name="base_link">
-      <visual>
-        <geometry>
-          <!-- new mesh -->
-          <mesh filename="file://$(find kobuki_description)/meshes/main_body.dae" />
-        </geometry>
-        <origin xyz="0.001 0 0.05199" rpy="0 0 0"/>
-      </visual>
-      <collision name="base">
-        <geometry>
-          <cylinder length="0.10938" radius="0.178"/>
-        </geometry>
-        <origin xyz="0.0 0 0.05949" rpy="0 0 0"/>
-      </collision>
-      <inertial>
-        <!-- COM experimentally determined -->
-        <origin xyz="0.01 0 0"/>
-        <mass value="2.4"/> <!-- 2.4/2.6 kg for small/big battery pack -->
-        <!-- Kobuki's inertia tensor is approximated by a cylinder with homogeneous mass distribution
-             More details http://en.wikipedia.org/wiki/List_of_moment_of_inertia_tensors
-             m = 2.4 kg; h = 0.09 m; r = 0.175 m
-             ixx = 1/12 * m * (3 * r^2 + h^2)
-             iyy = 1/12 * m * (3 * r^2 + h^2)
-             izz = 1/2 * m * r^2
-          -->
-        <inertia ixx="0.019995" ixy="0.0" ixz="0.0"
-                 iyy="0.019995" iyz="0.0"
-                 izz="0.03675" />
-      </inertial>
-    </link>
-    <joint name="wheel_left_joint" type="continuous">
-      <parent link="base_link"/>
-      <child link="wheel_left_link"/>
-      <origin xyz="0.00 ${0.23/2} 0.0250" rpy="${-M_PI/2} 0 0"/>
-      <axis xyz="0 0 1"/>
-    </joint>
-    <link name="wheel_left_link">
-      <visual>
-        <geometry>
-          <mesh filename="file://$(find kobuki_description)/meshes/wheel.dae"/>
-        </geometry>
-        <origin xyz="0 0 0" rpy="0 0 0"/>
-      </visual>
-      <collision>
-        <geometry>
-          <cylinder length="0.0206" radius="0.035"/>
-        </geometry>
-        <origin rpy="0 0 0" xyz="0 0 0"/>
-      </collision>
-      <inertial>
-        <mass value="0.01" />
-        <origin xyz="0 0 0" />
-        <inertia ixx="0.001" ixy="0.0" ixz="0.0"
-                 iyy="0.001" iyz="0.0"
-                 izz="0.001" />
-      </inertial>
-    </link>
-    <joint name="wheel_right_joint" type="continuous">
-      <parent link="base_link"/>
-      <child link="wheel_right_link"/>
-      <origin xyz="0.00 -${0.23/2} 0.0250" rpy="${-M_PI/2} 0 0"/>
-      <axis xyz="0 0 1"/>
-    </joint>
-    <link name="wheel_right_link">
-      <visual>
-        <geometry>
-          <mesh filename="file://$(find kobuki_description)/meshes/wheel.dae"/>
-        </geometry>
-        <origin xyz="0 0 0" rpy="0 0 0"/>
-      </visual>
-      <collision>
-        <geometry>
-          <cylinder length="0.0206" radius="0.035"/>
-        </geometry>
-        <origin rpy="0 0 0" xyz="0 0 0"/>
-      </collision>
-      <inertial>
-        <mass value="0.01" />
-        <origin xyz="0 0 0" />
-        <inertia ixx="0.001" ixy="0.0" ixz="0.0"
-                 iyy="0.001" iyz="0.0"
-                 izz="0.001" />
-      </inertial>
-    </link>
-    <joint name="caster_front_joint" type="fixed">
-      <parent link="base_link"/>
-      <child link="caster_front_link"/>
-      <origin xyz="0.115 0.0 0.007" rpy="${-M_PI/2} 0 0"/>
-    </joint>
-    <link name="caster_front_link">
-      <collision>
-        <geometry>
-          <cylinder length="0.0176" radius="0.017"/>
-        </geometry>
-        <origin rpy="0 0 0" xyz="0 0 0"/>
-      </collision>
-      <inertial>
-        <mass value="0.01" />
-        <origin xyz="0 0 0" />
-        <inertia ixx="0.001" ixy="0.0" ixz="0.0"
-                 iyy="0.001" iyz="0.0"
-                 izz="0.001" />
-      </inertial>
-    </link>
-    <joint name="caster_back_joint" type="fixed">
-      <parent link="base_link"/>
-      <child link="caster_back_link"/>
-      <origin xyz="-0.135 0.0 0.009" rpy="${-M_PI/2} 0 0"/>
-    </joint>
-    <link name="caster_back_link">
-      <collision>
-        <geometry>
-          <cylinder length="0.0176" radius="0.017"/>
-        </geometry>
-        <origin rpy="0 0 0" xyz="0 0 0"/>
-      </collision>
-      <inertial>
-        <mass value="0.01" />
-        <origin xyz="0 0 0" />
-        <inertia ixx="0.001" ixy="0.0" ixz="0.0"
-                 iyy="0.001" iyz="0.0"
-                 izz="0.001" />
-      </inertial>
-    </link>
-    <!-- Kobuki's sensors -->
-    <joint name="gyro_joint" type="fixed">
-      <axis xyz="0 1 0"/>
-      <origin xyz="0.056 0.062 0.0202" rpy="0 0 0"/>
-      <parent link="base_link"/>
-      <child link="gyro_link"/>
-    </joint>
-    <link name="gyro_link">
-      <inertial>
-        <mass value="0.001"/>
-        <origin xyz="0 0 0" rpy="0 0 0"/>
-        <inertia ixx="0.0001" ixy="0" ixz="0"
-                 iyy="0.000001" iyz="0"
-                 izz="0.0001"/>
-      </inertial>
-    </link>
-    <joint name="cliff_sensor_left_joint" type="fixed">
-      <origin xyz="0.08734 0.13601 0.0214" rpy="0 ${M_PI/2} 0" />
-      <parent link="base_link"/>
-      <child link="cliff_sensor_left_link" />
-    </joint>
-    <link name="cliff_sensor_left_link">
-      <inertial>
-        <mass value="0.0001" />
-        <origin xyz="0 0 0" />
-        <inertia ixx="0.0001" ixy="0.0" ixz="0.0"
-                 iyy="0.0001" iyz="0.0"
-                 izz="0.0001" />
-      </inertial>
-    </link>
-    <joint name="cliff_sensor_right_joint" type="fixed">
-      <origin xyz="0.085 -0.13601 0.0214" rpy="0 ${M_PI/2} 0" />
-      <parent link="base_link"/>
-      <child link="cliff_sensor_right_link" />
-    </joint>
-    <link name="cliff_sensor_right_link">
-      <inertial>
-        <mass value="0.0001" />
-        <origin xyz="0 0 0" />
-        <inertia ixx="0.0001" ixy="0.0" ixz="0.0"
-                 iyy="0.0001" iyz="0.0"
-                 izz="0.0001" />
-      </inertial>
-    </link>
-    <joint name="cliff_sensor_front_joint" type="fixed">
-      <origin xyz="0.156 0.00 0.0214" rpy="0 ${M_PI/2} 0" />
-      <parent link="base_link"/>
-      <child link="cliff_sensor_front_link" />
-    </joint>
-    <link name="cliff_sensor_front_link">
-      <inertial>
-        <mass value="0.0001" />
-        <origin xyz="0 0 0" />
-        <inertia ixx="0.0001" ixy="0.0" ixz="0.0"
-                 iyy="0.0001" iyz="0.0"
-                 izz="0.0001" />
-      </inertial>
-    </link>
-    <gazebo>
-      <plugin filename="gz-sim-diff-drive-system" name="gz::sim::systems::DiffDrive">
-        <!-- Remove <ros> tag. -->
-        <!-- wheels -->
-        <left_joint>wheel_left_joint</left_joint>
-        <right_joint>wheel_right_joint</right_joint>
-        <!-- kinematics -->
-        <wheel_separation>0.223087</wheel_separation>
-        <wheel_radius>0.035</wheel_radius> <!-- computed from <wheel_diameter> in the original plugin-->
-        <!-- limits -->
-        <max_linear_acceleration>1.0</max_linear_acceleration> <!-- computed from <max_linear_acceleration> in the original plugin-->
-        <topic>cmd_vel</topic> <!-- from <commant_topic> -->
-        <child_frame_id>base_footprint</child_frame_id> <!-- from <robot_base_frame> -->
-        <odom_publisher_frequency>30</odom_publisher_frequency> <!-- from <update_rate>-->
-        <tf_topic>/tf</tf_topic> <!-- Short topic name for tf output -->
-      </plugin>
-    </gazebo>
-     <gazebo reference="camera_link">
-  <sensor name="camera" type="depth">
-    <update_rate>30</update_rate>
-    <camera>
-      <horizontal_fov>1.047198</horizontal_fov>
-      <image>
-        <width>640</width>
-        <height>480</height>
-        <format>B8G8R8</format>
-      </image>
-      <clip>
-        <near>0.05</near>
-        <far>3</far>
-      </clip>
-    </camera>
-    <!-- <plugin name="camera_controller" filename="libgazebo_ros_camera.so">
-      <baseline>0.2</baseline>
-      <alwaysOn>true</alwaysOn>
-      <updateRate>1.0</updateRate>
-      <frame_Name>camera_link</frame_Name>
-      <pointCloudCutoff>0.5</pointCloudCutoff>
-      <pointCloudCutoffMax>3.0</pointCloudCutoffMax>
-      <distortionK1>0.00000001</distortionK1>
-      <distortionK2>0.00000001</distortionK2>
-      <distortionK3>0.00000001</distortionK3>
-      <distortionT1>0.00000001</distortionT1>
-      <distortionT2>0.00000001</distortionT2>
-      <CxPrime>0</CxPrime>
-      <Cx>0</Cx>
-      <Cy>0</Cy>
-      <focalLength>0</focalLength>
-      <hackBaseline>0</hackBaseline>
-    </plugin> -->
-  </sensor>
-</gazebo>
-<joint name="laser_joint" type="fixed">
-      <origin xyz="0.0 0.0 0.37" rpy="0 0 0" />
-      <parent link="base_link"/>
-      <child link="laser_link" />
-    </joint>
-<link name="laser_link">
-	<visual>
-        <geometry>
-          <mesh filename="file://$(find kobuki_description)/meshes/sensors/rplidar.dae" scale="0.001 0.001 0.001" />
-        </geometry>
-        <origin xyz="0 0 0.025" rpy="-1.5707 0 -1.5707"/>
-      </visual>
-      <inertial>
-        <mass value="0.0001" />
-        <origin xyz="0 0 0" />
-        <inertia ixx="0.0001" ixy="0.0" ixz="0.0"
-                 iyy="0.0001" iyz="0.0"
-                 izz="0.0001" />
-      </inertial>
-    </link>
-  <gazebo reference="laser_link">
-    <sensor name="lidar" type="ray">
-      <always_on>true</always_on>
-      <visualize>true</visualize>
-      <update_rate>5</update_rate>
-      <ray>
-        <scan>
-          <horizontal>
-            <samples>360</samples>
-            <resolution>1.000000</resolution>
-            <min_angle>0.000000</min_angle>
-            <max_angle>6.280000</max_angle>
-          </horizontal>
-        </scan>
-        <range>
-          <min>0.17</min>
-          <max>3.5</max>
-          <resolution>0.015000</resolution>
-        </range>
-        <noise>
-          <type>gaussian</type>
-          <mean>0.0</mean>
-          <stddev>0.01</stddev>
-        </noise>
-      </ray>
-      <!-- <plugin filename="libgazebo_ros_ray_sensor.so" name="scan">
-        <ros>
-          <remapping>~/out:=scan</remapping>
-        </ros>
-        <output_type>sensor_msgs/LaserScan</output_type>
-        <frame_name>laser_link</frame_name>
-      </plugin> -->
-    </sensor>
+<robot name="kobuki_gazebo" xmlns:xacro="http://ros.org/wiki/xacro">
+  <xacro:macro name="kobuki_gazebo" params="lidar camera">
+  <gazebo>
+    <plugin filename="gz-sim-diff-drive-system" name="gz::sim::systems::DiffDrive">
+      <left_joint>wheel_left_joint</left_joint>
+      <right_joint>wheel_right_joint</right_joint>
+      <wheel_separation>0.223087</wheel_separation>
+      <wheel_radius>0.035</wheel_radius>
+      <max_linear_acceleration>1.0</max_linear_acceleration>
+      <topic>cmd_vel</topic>
+      <child_frame_id>base_footprint</child_frame_id>
+      <odom_publisher_frequency>30</odom_publisher_frequency>
+      <tf_topic>/tf</tf_topic>
+    </plugin>
   </gazebo>
+    <xacro:if value="$(arg lidar)">
+        <sensor name="kobuki_lidar" type="gpu_lidar">
+            <always_on>true</always_on>
+            <visualize>true</visualize>
+            <pose>0 0 0 0 0 0</pose>
+            <update_rate>5</update_rate>
+            <topic>scan_raw</topic>
+            <gz_frame_id>laser_link</gz_frame_id>
+            <lidar>
+                <ray>
+                    <scan>
+                      <horizontal>
+                        <samples>360</samples>
+                        <resolution>1.000000</resolution>
+                        <min_angle>0.000000</min_angle>
+                        <max_angle>6.280000</max_angle>
+                      </horizontal>
+                    </scan>
+                    <range>
+                      <min>0.17</min>
+                      <max>3.5</max>
+                      <resolution>0.015000</resolution>
+                    </range>
+                    <noise>
+                      <type>gaussian</type>
+                      <mean>0.0</mean>
+                      <stddev>0.01</stddev>
+                    </noise>
+                  </ray>
+            </lidar>
+          </sensor>
+    </xacro:if>
+    <!-- <xacro:if value="$(camera)">
+    </xacro:if> -->
   </xacro:macro>
 </robot>

File: kobuki_description/urdf/sensors/asus_xtion_pro.urdf.xacro (robot description, xacro)
@@ -1,5 +1,4 @@
 <?xml version="1.0"?>
 <robot name="sensor_asus_xtion_pro" xmlns:xacro="http://ros.org/wiki/xacro">
-  <xacro:include filename="$(find kobuki_description)/urdf/turtlebot_gazebo.urdf.xacro"/>
   <xacro:include filename="$(find kobuki_description)/urdf/turtlebot_properties.urdf.xacro"/>
   <!-- Xacro properties -->
@@ -62,33 +61,4 @@
     </joint>
     <link name="camera_depth_optical_frame"/>
-    <!-- RGBD sensor for simulation, same as Kinect -->
-    <turtlebot_sim_3dsensor/>
-    <!-- Asus mount -->
-    <joint name="mount_asus_xtion_pro_joint" type="fixed">
-      <origin xyz="-0.1024 0.0 0.272" rpy="0 0 0"/>
-      <parent link="${parent}"/>
-      <child link="mount_asus_xtion_pro_link"/>
-    </joint>
-    <link name="mount_asus_xtion_pro_link">
-      <visual>
-        <origin xyz="0 0 0" rpy="${-M_PI/2} 0 0"/>
-        <geometry>
-          <mesh filename="file://$(find kobuki_description)/meshes/sensors/xtion_pro_stack.dae"/>
-        </geometry>
-      </visual>
-      <collision>
-        <origin xyz="0.0 0.0 0.0" rpy="0 0 0" />
-        <geometry>
-        <box size="0.0330 0.2760 0.0120"/>
-      </geometry>
-      </collision>
-      <inertial>
-        <mass value="0.170" />
-        <origin xyz="0 0 0" />
-        <inertia ixx="0.001152600" ixy="0.0" ixz="0.0"
-                 iyy="0.000148934" iyz="0.0"
-                 izz="0.001154654" />
-      </inertial>
-    </link>
   </xacro:macro>
 </robot>

File: kobuki_description/urdf/turtlebot_properties.urdf.xacro (robot description, xacro)
@@ -19,7 +19,7 @@
      (currently in development and awaiting feedback)
    -->
-	<xacro:property name="cam_px" value="-0.087" />
+	<xacro:property name="cam_px" value="0.087" />
 <!--	<xacro:property name="cam_py" value="-0.0125" /> Y varies for different configurations. get sets in sensors_urdf -->
-	<xacro:property name="cam_pz" value="0.2870" />
+	<xacro:property name="cam_pz" value="0.21" />
 	<xacro:property name="cam_or" value="0" />
 	<xacro:property name="cam_op" value="0" />

Commit message: prefix added to cmd_vel in gazebo topics, trying to discover how to modify de yaml bridge for multirobot

File: kobuki_description/urdf/kobuki.urdf.xacro (robot description, xacro)
@@ -9,4 +9,5 @@
   <xacro:arg name="camera" default="false" />
   <xacro:arg name="structure" default="false" />
+  <xacro:arg name="prefix" default="false" />
   <xacro:arg name="gazebo" default="false" />
   <xacro:include filename="$(find kobuki_description)/urdf/kobuki_base.urdf.xacro" />
@@ -42,5 +43,5 @@
   <xacro:if value="$(arg gazebo)">
     <xacro:include filename="$(find kobuki_description)/urdf/kobuki_gazebo.urdf.xacro"/>
-    <xacro:kobuki_gazebo lidar="$(arg lidar)" camera="$(arg camera)"/>
+    <xacro:kobuki_gazebo lidar="$(arg lidar)" camera="$(arg camera)" prefix="$(arg prefix)"/>
   </xacro:if>
 </robot>

File: kobuki_description/urdf/kobuki_gazebo.urdf.xacro (robot description, xacro)
@@ -1,5 +1,5 @@
 <?xml version="1.0" ?>
 <robot name="kobuki_gazebo" xmlns:xacro="http://ros.org/wiki/xacro">
-  <xacro:macro name="kobuki_gazebo" params="lidar camera">
+  <xacro:macro name="kobuki_gazebo" params="lidar camera prefix">
     <gazebo>
       <plugin filename="gz-sim-diff-drive-system" name="gz::sim::systems::DiffDrive">
@@ -9,10 +9,10 @@
         <wheel_radius>0.035</wheel_radius>
         <max_linear_acceleration>1.0</max_linear_acceleration>
-        <topic>cmd_vel</topic>
+        <topic>$(arg prefix)/cmd_vel</topic>
         <odom_topic>odom</odom_topic>
         <frame_id>odom</frame_id>
         <child_frame_id>base_footprint</child_frame_id>
         <odom_publisher_frequency>30</odom_publisher_frequency>
-        <tf_topic>/tf</tf_topic>
+        <tf_topic>$(arg prefix)/tf</tf_topic>
       </plugin>
       <plugin filename="gz-sim-joint-state-publisher-system" name="gz::sim::systems::JointStatePublisher">
