Commit message: tf tree fixed with namespaces, error in joint_state_publisher unable to receive robot_description

File: kobuki_description/urdf/kobuki.urdf.xacro (robot description, xacro)
@@ -9,39 +9,39 @@
   <xacro:arg name="camera" default="false" />
   <xacro:arg name="structure" default="false" />
-  <xacro:arg name="prefix" default="" />
+  <xacro:arg name="namespace" default="" />
   <xacro:arg name="gazebo" default="false" />
   <xacro:include filename="$(find kobuki_description)/urdf/kobuki_base.urdf.xacro" />
   <xacro:include filename="$(find kobuki_description)/urdf/turtlebot_common_library.urdf.xacro" />
-  <xacro:kobuki_base/>
+  <xacro:kobuki_base namespace="$(arg namespace)"/>
   <xacro:if value="$(arg structure)">
     <xacro:include filename="$(find kobuki_description)/urdf/stacks/hexagons.urdf.xacro"/>
     <xacro:include filename="$(find kobuki_description)/urdf/stacks/circles.urdf.xacro"/>
-    <xacro:stack_hexagons parent="base_link"/>
-    <xacro:turtlebot_standoff_1in number="0" parent="base_link" x_loc="0.120" y_loc="0.082" z_loc="0.09"/>
-    <xacro:turtlebot_standoff_1in number="1" parent="base_link" x_loc="0.055" y_loc="0.120" z_loc="0.09"/>
-    <xacro:turtlebot_standoff_1in number="2" parent="base_link" x_loc="-0.055" y_loc="0.120" z_loc="0.09"/>
-    <xacro:turtlebot_standoff_1in number="3" parent="base_link" x_loc="0.120" y_loc="-0.082" z_loc="0.09"/>
-    <xacro:turtlebot_standoff_1in number="4" parent="base_link" x_loc="0.055" y_loc="-0.120" z_loc="0.09"/>
-    <xacro:turtlebot_standoff_1in number="5" parent="base_link" x_loc="-0.055" y_loc="-0.120" z_loc="0.09"/>
-    <xacro:turtlebot_standoff_2in number="0" parent="base_link" x_loc="0.0381" y_loc="0.1505" z_loc="0.1340"/>
-    <xacro:turtlebot_standoff_2in number="1" parent="base_link" x_loc="0.0381" y_loc="-0.1505" z_loc="0.1340"/>
-    <xacro:turtlebot_standoff_2in number="2" parent="base_link" x_loc="-0.0381" y_loc="0.1505" z_loc="0.1340"/>
-    <xacro:turtlebot_standoff_2in number="3" parent="base_link" x_loc="-0.0381" y_loc="-0.1505" z_loc="0.1340"/>
-    <xacro:turtlebot_standoff_8in number="0" parent="base_link" x_loc="0.0381" y_loc="0.1505" z_loc="0.1900"/>
-    <xacro:turtlebot_standoff_8in number="1" parent="base_link" x_loc="0.0381" y_loc="-0.1505" z_loc="0.1900"/>
-    <xacro:turtlebot_standoff_8in number="2" parent="base_link" x_loc="-0.0381" y_loc="0.1505" z_loc="0.1900"/>
-    <xacro:turtlebot_standoff_8in number="3" parent="base_link" x_loc="-0.0381" y_loc="-0.1505" z_loc="0.1900"/>
+    <xacro:stack_hexagons parent="$(arg namespace)/base_link" namespace="$(arg namespace)"/>
+    <xacro:turtlebot_standoff_1in number="0" parent="$(arg namespace)/base_link" x_loc="0.120" y_loc="0.082" z_loc="0.09" namespace="$(arg namespace)"/>
+    <xacro:turtlebot_standoff_1in number="1" parent="$(arg namespace)/base_link" x_loc="0.055" y_loc="0.120" z_loc="0.09" namespace="$(arg namespace)"/>
+    <xacro:turtlebot_standoff_1in number="2" parent="$(arg namespace)/base_link" x_loc="-0.055" y_loc="0.120" z_loc="0.09" namespace="$(arg namespace)"/>
+    <xacro:turtlebot_standoff_1in number="3" parent="$(arg namespace)/base_link" x_loc="0.120" y_loc="-0.082" z_loc="0.09" namespace="$(arg namespace)"/>
+    <xacro:turtlebot_standoff_1in number="4" parent="$(arg namespace)/base_link" x_loc="0.055" y_loc="-0.120" z_loc="0.09" namespace="$(arg namespace)"/>
+    <xacro:turtlebot_standoff_1in number="5" parent="$(arg namespace)/base_link" x_loc="-0.055" y_loc="-0.120" z_loc="0.09" namespace="$(arg namespace)"/>
+    <xacro:turtlebot_standoff_2in number="0" parent="$(arg namespace)/base_link" x_loc="0.0381" y_loc="0.1505" z_loc="0.1340" namespace="$(arg namespace)"/>
+    <xacro:turtlebot_standoff_2in number="1" parent="$(arg namespace)/base_link" x_loc="0.0381" y_loc="-0.1505" z_loc="0.1340" namespace="$(arg namespace)"/>
+    <xacro:turtlebot_standoff_2in number="2" parent="$(arg namespace)/base_link" x_loc="-0.0381" y_loc="0.1505" z_loc="0.1340" namespace="$(arg namespace)"/>
+    <xacro:turtlebot_standoff_2in number="3" parent="$(arg namespace)/base_link" x_loc="-0.0381" y_loc="-0.1505" z_loc="0.1340" namespace="$(arg namespace)"/>
+    <xacro:turtlebot_standoff_8in number="0" parent="$(arg namespace)/base_link" x_loc="0.0381" y_loc="0.1505" z_loc="0.1900" namespace="$(arg namespace)"/>
+    <xacro:turtlebot_standoff_8in number="1" parent="$(arg namespace)/base_link" x_loc="0.0381" y_loc="-0.1505" z_loc="0.1900" namespace="$(arg namespace)"/>
+    <xacro:turtlebot_standoff_8in number="2" parent="$(arg namespace)/base_link" x_loc="-0.0381" y_loc="0.1505" z_loc="0.1900" namespace="$(arg namespace)"/>
+    <xacro:turtlebot_standoff_8in number="3" parent="$(arg namespace)/base_link" x_loc="-0.0381" y_loc="-0.1505" z_loc="0.1900" namespace="$(arg namespace)"/>
   </xacro:if>
   <xacro:if value="$(arg lidar)">
     <xacro:include filename="$(find kobuki_description)/urdf/sensors/lidar.urdf.xacro"/>
-    <xacro:sensor_lidar/>
+    <xacro:sensor_lidar namespace="$(arg namespace)"/>
   </xacro:if>
   <xacro:if value="$(arg camera)">
     <xacro:include filename="$(find kobuki_description)/urdf/sensors/asus_xtion_pro.urdf.xacro"/>
-    <xacro:sensor_asus_xtion_pro parent="base_link"/>
+    <xacro:sensor_asus_xtion_pro parent="$(arg namespace)/base_link"/>
   </xacro:if>
   <xacro:if value="$(arg gazebo)">
     <xacro:include filename="$(find kobuki_description)/urdf/kobuki_gazebo.urdf.xacro"/>
-    <xacro:kobuki_gazebo lidar="$(arg lidar)" camera="$(arg camera)" prefix="$(arg prefix)"/>
+    <xacro:kobuki_gazebo lidar="$(arg lidar)" camera="$(arg camera)" namespace="$(arg namespace)"/>
   </xacro:if>
 </robot>

File: kobuki_description/urdf/kobuki_base.urdf.xacro (robot description, xacro)
@@ -9,6 +9,6 @@
   <xacro:include filename="$(find kobuki_description)/urdf/common_properties.urdf.xacro"/>
   <!-- Kobuki -->
-  <xacro:macro name="kobuki_base">
-    <link name="base_footprint"/>
+  <xacro:macro name="kobuki_base" params = "namespace">
+    <link name="$(arg namespace)/base_footprint"/>
     <!--
        Base link is set at the bottom of the base mould.
@@ -20,10 +20,10 @@
        to 0.352.
       -->
-    <joint name="base_joint" type="fixed">
+    <joint name="$(arg namespace)/base_joint" type="fixed">
       <origin xyz="0 0 0.0102" rpy="0 0 0" />
-      <parent link="base_footprint"/>
-      <child link="base_link" />
-    </joint>
-    <link name="base_link">
+      <parent link="$(arg namespace)/base_footprint"/>
+      <child link="$(arg namespace)/base_link" />
+    </joint>
+    <link name="$(arg namespace)/base_link">
       <visual>
         <geometry>
@@ -55,11 +55,11 @@
       </inertial>
     </link>
-    <joint name="wheel_left_joint" type="continuous">
-      <parent link="base_link"/>
-      <child link="wheel_left_link"/>
+    <joint name="$(arg namespace)/wheel_left_joint" type="continuous">
+      <parent link="$(arg namespace)/base_link"/>
+      <child link="$(arg namespace)/wheel_left_link"/>
       <origin xyz="0.00 ${0.23/2} 0.0250" rpy="${-M_PI/2} 0 0"/>
       <axis xyz="0 0 1"/>
     </joint>
-    <link name="wheel_left_link">
+    <link name="$(arg namespace)/wheel_left_link">
       <visual>
         <geometry>
@@ -82,11 +82,11 @@
       </inertial>
     </link>
-    <joint name="wheel_right_joint" type="continuous">
-      <parent link="base_link"/>
-      <child link="wheel_right_link"/>
+    <joint name="$(arg namespace)/wheel_right_joint" type="continuous">
+      <parent link="$(arg namespace)/base_link"/>
+      <child link="$(arg namespace)/wheel_right_link"/>
       <origin xyz="0.00 -${0.23/2} 0.0250" rpy="${-M_PI/2} 0 0"/>
       <axis xyz="0 0 1"/>
     </joint>
-    <link name="wheel_right_link">
+    <link name="$(arg namespace)/wheel_right_link">
       <visual>
         <geometry>
@@ -109,10 +109,10 @@
       </inertial>
     </link>
-    <joint name="caster_front_joint" type="fixed">
-      <parent link="base_link"/>
-      <child link="caster_front_link"/>
+    <joint name="$(arg namespace)/caster_front_joint" type="fixed">
+      <parent link="$(arg namespace)/base_link"/>
+      <child link="$(arg namespace)/caster_front_link"/>
       <origin xyz="0.115 0.0 0.007" rpy="${-M_PI/2} 0 0"/>
     </joint>
-    <link name="caster_front_link">
+    <link name="$(arg namespace)/caster_front_link">
       <collision>
         <geometry>
@@ -129,10 +129,10 @@
       </inertial>
     </link>
-    <joint name="caster_back_joint" type="fixed">
-      <parent link="base_link"/>
-      <child link="caster_back_link"/>
+    <joint name="$(arg namespace)/caster_back_joint" type="fixed">
+      <parent link="$(arg namespace)/base_link"/>
+      <child link="$(arg namespace)/caster_back_link"/>
       <origin xyz="-0.135 0.0 0.009" rpy="${-M_PI/2} 0 0"/>
     </joint>
-    <link name="caster_back_link">
+    <link name="$(arg namespace)/caster_back_link">
       <collision>
         <geometry>
@@ -150,11 +150,11 @@
     </link>
     <!-- Kobuki's sensors -->
-    <joint name="gyro_joint" type="fixed">
+    <joint name="$(arg namespace)/gyro_joint" type="fixed">
       <axis xyz="0 1 0"/>
       <origin xyz="0.056 0.062 0.0202" rpy="0 0 0"/>
-      <parent link="base_link"/>
-      <child link="gyro_link"/>
-    </joint>
-    <link name="gyro_link">
+      <parent link="$(arg namespace)/base_link"/>
+      <child link="$(arg namespace)/gyro_link"/>
+    </joint>
+    <link name="$(arg namespace)/gyro_link">
       <inertial>
         <mass value="0.001"/>
@@ -165,10 +165,10 @@
       </inertial>
     </link>
-    <joint name="cliff_sensor_left_joint" type="fixed">
+    <joint name="$(arg namespace)/cliff_sensor_left_joint" type="fixed">
       <origin xyz="0.08734 0.13601 0.0214" rpy="0 ${M_PI/2} 0" />
-      <parent link="base_link"/>
-      <child link="cliff_sensor_left_link" />
-    </joint>
-    <link name="cliff_sensor_left_link">
+      <parent link="$(arg namespace)/base_link"/>
+      <child link="$(arg namespace)/cliff_sensor_left_link" />
+    </joint>
+    <link name="$(arg namespace)/cliff_sensor_left_link">
       <inertial>
         <mass value="0.0001" />
@@ -179,10 +179,10 @@
       </inertial>
     </link>
-    <joint name="cliff_sensor_right_joint" type="fixed">
+    <joint name="$(arg namespace)/cliff_sensor_right_joint" type="fixed">
       <origin xyz="0.085 -0.13601 0.0214" rpy="0 ${M_PI/2} 0" />
-      <parent link="base_link"/>
-      <child link="cliff_sensor_right_link" />
-    </joint>
-    <link name="cliff_sensor_right_link">
+      <parent link="$(arg namespace)/base_link"/>
+      <child link="$(arg namespace)/cliff_sensor_right_link" />
+    </joint>
+    <link name="$(arg namespace)/cliff_sensor_right_link">
       <inertial>
         <mass value="0.0001" />
@@ -193,10 +193,10 @@
       </inertial>
     </link>
-    <joint name="cliff_sensor_front_joint" type="fixed">
+    <joint name="$(arg namespace)/cliff_sensor_front_joint" type="fixed">
       <origin xyz="0.156 0.00 0.0214" rpy="0 ${M_PI/2} 0" />
-      <parent link="base_link"/>
-      <child link="cliff_sensor_front_link" />
-    </joint>
-    <link name="cliff_sensor_front_link">
+      <parent link="$(arg namespace)/base_link"/>
+      <child link="$(arg namespace)/cliff_sensor_front_link" />
+    </joint>
+    <link name="$(arg namespace)/cliff_sensor_front_link">
       <inertial>
         <mass value="0.0001" />

File: kobuki_description/urdf/kobuki_gazebo.urdf.xacro (robot description, xacro)
@@ -1,5 +1,5 @@
 <?xml version="1.0" ?>
 <robot name="kobuki_gazebo" xmlns:xacro="http://ros.org/wiki/xacro">
-  <xacro:macro name="kobuki_gazebo" params="lidar camera prefix">
+  <xacro:macro name="kobuki_gazebo" params="lidar camera namespace">
     <gazebo>
       <plugin filename="gz-sim-diff-drive-system" name="gz::sim::systems::DiffDrive">
@@ -9,13 +9,13 @@
         <wheel_radius>0.035</wheel_radius>
         <max_linear_acceleration>1.0</max_linear_acceleration>
-        <topic>$(arg prefix)/cmd_vel</topic>
-        <odom_topic>$(arg prefix)/odom</odom_topic>
+        <topic>$(arg namespace)/cmd_vel</topic>
+        <odom_topic>$(arg namespace)/odom</odom_topic>
         <frame_id>odom</frame_id>
         <child_frame_id>base_footprint</child_frame_id>
         <odom_publisher_frequency>30</odom_publisher_frequency>
-        <tf_topic>$(arg prefix)/tf</tf_topic>
+        <tf_topic>/tf</tf_topic>
       </plugin>
       <plugin filename="gz-sim-joint-state-publisher-system" name="gz::sim::systems::JointStatePublisher">
-        <topic>$(arg prefix)/joint_states</topic>
+        <topic>$(arg namespace)/joint_states</topic>
         <joint>wheel_left_joint</joint>
         <joint>wheel_right_joint</joint>
@@ -33,5 +33,5 @@
             <visualize>true</visualize>
             <update_rate>5</update_rate>
-            <topic>$(arg prefix)/scan_raw</topic>
+            <topic>$(arg namespace)/scan_raw</topic>
             <gz_frame_id>laser_link</gz_frame_id>
             <lidar>
@@ -64,5 +64,5 @@
           <update_rate>30.0</update_rate>
           <visualize>true</visualize>
-          <topic>$(arg prefix)/rgbd_camera</topic>
+          <topic>$(arg namespace)/rgbd_camera</topic>
           <camera>
             <horizontal_fov>${63.0*M_PI/180.0}</horizontal_fov>

File: kobuki_description/urdf/sensors/lidar.urdf.xacro (robot description, xacro)
@@ -1,6 +1,6 @@
 <?xml version="1.0"?>
 <robot name="sensor_lidar" xmlns:xacro="http://ros.org/wiki/xacro">
-  <xacro:macro name="sensor_lidar">
-  <link name="laser_link">
+  <xacro:macro name="sensor_lidar" params = "namespace">
+  <link name="$(arg namespace)/laser_link">
       <visual>
           <geometry>
@@ -17,8 +17,8 @@
         </inertial>
       </link>
-      <joint name="laser_joint" type="fixed">
+      <joint name="$(arg namespace)/laser_joint" type="fixed">
         <origin xyz="0.0 0.0 0.37" rpy="0 0 0" />
-        <parent link="base_link"/>
-        <child link="laser_link" />
+        <parent link="$(arg namespace)/base_link"/>
+        <child link="$(arg namespace)/laser_link" />
     </joint>
   </xacro:macro>

File: kobuki_description/urdf/stacks/circles.urdf.xacro (robot description, xacro)
@@ -1,5 +1,5 @@
 <?xml version="1.0"?>
 <robot name="turtlebot_hardware" xmlns:xacro="http://ros.org/wiki/xacro">
-  <xacro:macro name="turtlebot_spacer" params="parent number x_loc y_loc z_loc">
+  <xacro:macro name="turtlebot_spacer" params="parent number x_loc y_loc z_loc namespace">
     <joint name="spacer_${number}_joint" type="fixed">
       <origin xyz="${x_loc} ${y_loc} ${z_loc}" rpy="0 0 0" />
@@ -29,11 +29,11 @@
     </link>
   </xacro:macro>
-  <xacro:macro name="turtlebot_standoff_1in" params="parent number x_loc y_loc z_loc">
-    <joint name="standoff_1in_${number}_joint" type="fixed">
-      <origin xyz="${x_loc} ${y_loc} ${z_loc}" rpy="0 0 0" />
-      <parent link="${parent}"/>
-      <child link="standoff_1in_${number}_link" />
-    </joint>
-    <link name="standoff_1in_${number}_link">
+  <xacro:macro name="turtlebot_standoff_1in" params="parent number x_loc y_loc z_loc namespace">
+    <joint name="$(arg namespace)/standoff_1in_${number}_joint" type="fixed">
+      <origin xyz="${x_loc} ${y_loc} ${z_loc}" rpy="0 0 0" />
+      <parent link="${parent}"/>
+      <child link="$(arg namespace)/standoff_1in_${number}_link" />
+    </joint>
+    <link name="$(arg namespace)/standoff_1in_${number}_link">
       <inertial>
         <mass value="0.001" />
@@ -57,11 +57,11 @@
     </link>
   </xacro:macro>
-  <xacro:macro name="turtlebot_standoff_2in" params="parent number x_loc y_loc z_loc">
-    <joint name="standoff_2in_${number}_joint" type="fixed">
-      <origin xyz="${x_loc} ${y_loc} ${z_loc}" rpy="0 0 0" />
-      <parent link="${parent}"/>
-      <child link="standoff_2in_${number}_link" />
-    </joint>
-    <link name="standoff_2in_${number}_link">
+  <xacro:macro name="turtlebot_standoff_2in" params="parent number x_loc y_loc z_loc namespace">
+    <joint name="$(arg namespace)/standoff_2in_${number}_joint" type="fixed">
+      <origin xyz="${x_loc} ${y_loc} ${z_loc}" rpy="0 0 0" />
+      <parent link="${parent}"/>
+      <child link="$(arg namespace)/standoff_2in_${number}_link" />
+    </joint>
+    <link name="$(arg namespace)/standoff_2in_${number}_link">
       <inertial>
         <mass value="0.001" />
@@ -85,11 +85,11 @@
     </link>
   </xacro:macro>
-  <xacro:macro name="turtlebot_standoff_8in" params="parent number x_loc y_loc z_loc">
-    <joint name="standoff_8in_${number}_joint" type="fixed">
-      <origin xyz="${x_loc} ${y_loc} ${z_loc}" rpy="0 0 0" />
-      <parent link="${parent}"/>
-      <child link="standoff_8in_${number}_link" />
-    </joint>
-    <link name="standoff_8in_${number}_link">
+  <xacro:macro name="turtlebot_standoff_8in" params="parent number x_loc y_loc z_loc namespace">
+    <joint name="$(arg namespace)/standoff_8in_${number}_joint" type="fixed">
+      <origin xyz="${x_loc} ${y_loc} ${z_loc}" rpy="0 0 0" />
+      <parent link="${parent}"/>
+      <child link="$(arg namespace)/standoff_8in_${number}_link" />
+    </joint>
+    <link name="$(arg namespace)/standoff_8in_${number}_link">
       <inertial>
         <mass value="0.001" />
@@ -113,5 +113,5 @@
     </link>
   </xacro:macro>
-  <xacro:macro name="turtlebot_standoff_kinect" params="parent number x_loc y_loc z_loc">
+  <xacro:macro name="turtlebot_standoff_kinect" params="parent number x_loc y_loc z_loc namespace">
     <joint name="standoff_kinect_${number}_joint" type="fixed">
       <origin xyz="${x_loc} ${y_loc} ${z_loc}" rpy="0 0 0" />
@@ -141,5 +141,5 @@
     </link>
   </xacro:macro>
-  <xacro:macro name="stack_circles" params="parent">
+  <xacro:macro name="stack_circles" params="parent namespace">
     <turtlebot_spacer parent="${parent}" number="0" x_loc="-0.00254" y_loc="0.1114679" z_loc="0.062992"/>
     <turtlebot_spacer parent="${parent}" number="1" x_loc="-0.00254" y_loc="-0.1114679" z_loc="0.062992"/>

File: kobuki_description/urdf/stacks/hexagons.urdf.xacro (robot description, xacro)
@@ -9,5 +9,5 @@
   <!-- Xacro macros -->
   <!-- Pole macros -->
-  <xacro:macro name="stack_bottom_pole" params="parent number x_loc y_loc z_loc">
+  <xacro:macro name="stack_bottom_pole" params="parent number x_loc y_loc z_loc ">
     <joint name="pole_bottom_${number}_joint" type="fixed">
       <origin xyz="${x_loc} ${y_loc} ${z_loc}" rpy="0 0 0"/>
@@ -37,5 +37,5 @@
     </link>
   </xacro:macro>
-  <xacro:macro name="stack_middle_pole" params="parent number x_loc y_loc z_loc">
+  <xacro:macro name="stack_middle_pole" params="parent number x_loc y_loc z_loc ">
     <joint name="pole_middle_${number}_joint" type="fixed">
       <origin xyz="${x_loc} ${y_loc} ${z_loc}" rpy="0 0 0" />
@@ -65,5 +65,5 @@
     </link>
   </xacro:macro>
-  <xacro:macro name="stack_top_pole" params="parent number x_loc y_loc z_loc">
+  <xacro:macro name="stack_top_pole" params="parent number x_loc y_loc z_loc ">
     <joint name="pole_top_${number}_joint" type="fixed">
       <origin xyz="${x_loc} ${y_loc} ${z_loc}" rpy="0 0 0"/>
@@ -93,5 +93,5 @@
     </link>
   </xacro:macro>
-  <xacro:macro name="stack_3d_sensor_pole" params="parent number x_loc y_loc z_loc">
+  <xacro:macro name="stack_3d_sensor_pole" params="parent number x_loc y_loc z_loc ">
     <joint name="pole_kinect_${number}_joint" type="fixed">
       <origin xyz="${x_loc} ${y_loc} ${z_loc}" rpy="0 0 0"/>
@@ -126,5 +126,5 @@
     other, but there is no necessary reason to do so.
   -->
-  <xacro:macro name="stack_hexagons" params="parent">
+  <xacro:macro name="stack_hexagons" params="parent namespace">
     <stack_bottom_pole parent="${parent}" number="0" x_loc= "0.120" y_loc= "0.082" z_loc="0.1028"/>
     <stack_bottom_pole parent="${parent}" number="1" x_loc= "0.055" y_loc= "0.120" z_loc="0.1028"/>
@@ -133,10 +133,10 @@
     <stack_bottom_pole parent="${parent}" number="4" x_loc= "0.055" y_loc="-0.120" z_loc="0.1028"/>
     <stack_bottom_pole parent="${parent}" number="5" x_loc="-0.055" y_loc="-0.120" z_loc="0.1028"/>
-    <joint name="plate_bottom_joint" type="fixed">
+    <joint name="$(arg namespace)/plate_bottom_joint" type="fixed">
       <origin xyz="0.02364 0.0 0.1306" rpy="0 0 0"/>
       <parent link="${parent}"/>
-      <child link="plate_bottom_link"/>
-    </joint>
-    <link name="plate_bottom_link">
+      <child link="$(arg namespace)/plate_bottom_link"/>
+    </joint>
+    <link name="$(arg namespace)/plate_bottom_link">
       <visual>
         <origin xyz="0 0 0" rpy="0 0 0"/>
@@ -163,10 +163,10 @@
     <stack_middle_pole parent="${parent}" number="2" x_loc="-0.0381" y_loc= "0.1505" z_loc="0.1640"/>
     <stack_middle_pole parent="${parent}" number="3" x_loc="-0.0381" y_loc="-0.1505" z_loc="0.1640"/>
-    <joint name="plate_middle_joint" type="fixed">
+    <joint name="$(arg namespace)/plate_middle_joint" type="fixed">
       <origin xyz="-0.01364 0.0 0.1874" rpy="0 0 0"/>
       <parent link="${parent}"/>
-      <child link="plate_middle_link"/>
-    </joint>
-    <link name="plate_middle_link">
+      <child link="$(arg namespace)/plate_middle_link"/>
+    </joint>
+    <link name="$(arg namespace)/plate_middle_link">
       <visual>
         <origin xyz="0 0 0" rpy="0 0 0"/>
@@ -195,10 +195,10 @@
     <stack_3d_sensor_pole parent="${parent}" number="0" x_loc="-0.1024" y_loc= "0.098" z_loc="0.2372"/>
     <stack_3d_sensor_pole parent="${parent}" number="1" x_loc="-0.1024" y_loc="-0.098" z_loc="0.2372"/>
-    <joint name="plate_top_joint" type="fixed">
+    <joint name="$(arg namespace)/plate_top_joint" type="fixed">
       <origin xyz="-0.01364 0.0  0.3966" rpy="0 0 0"/>
       <parent link="${parent}"/>
-      <child link="plate_top_link"/>
-    </joint>
-    <link name="plate_top_link">
+      <child link="$(arg namespace)/plate_top_link"/>
+    </joint>
+    <link name="$(arg namespace)/plate_top_link">
       <visual>
         <origin xyz="0 0 0" rpy="0 0 0"/>
