Commit message: Bridge fixed with dynamic modification of the .yaml file, topics reviewed, and simulation running with two robots.

File: kobuki_description/urdf/kobuki.urdf.xacro (robot description, xacro)
@@ -5,5 +5,5 @@
     - 3d Sensor : kinect
 -->
-<robot name="kobuki" xmlns:xacro="http://ros.org/wiki/xacro" >
+<robot name="kobuki_$(arg namespace)" xmlns:xacro="http://ros.org/wiki/xacro" >
   <xacro:arg name="lidar" default="false" />
   <xacro:arg name="camera" default="false" />

File: kobuki_description/urdf/kobuki_gazebo.urdf.xacro (robot description, xacro)
@@ -4,6 +4,6 @@
     <gazebo>
       <plugin filename="gz-sim-diff-drive-system" name="gz::sim::systems::DiffDrive">
-        <left_joint>wheel_left_joint</left_joint>
-        <right_joint>wheel_right_joint</right_joint>
+        <left_joint>$(arg namespace)/wheel_left_joint</left_joint>
+        <right_joint>$(arg namespace)/wheel_right_joint</right_joint>
         <wheel_separation>0.223087</wheel_separation>
         <wheel_radius>0.035</wheel_radius>
@@ -12,5 +12,5 @@
         <odom_topic>$(arg namespace)/odom</odom_topic>
         <frame_id>odom</frame_id>
-        <child_frame_id>base_footprint</child_frame_id>
+        <child_frame_id>$(arg namespace)/base_footprint</child_frame_id>
         <odom_publisher_frequency>30</odom_publisher_frequency>
         <tf_topic>/tf</tf_topic>
@@ -18,6 +18,6 @@
       <plugin filename="gz-sim-joint-state-publisher-system" name="gz::sim::systems::JointStatePublisher">
         <topic>$(arg namespace)/joint_states</topic>
-        <joint>wheel_left_joint</joint>
-        <joint>wheel_right_joint</joint>
+        <joint>$(arg namespace)/wheel_left_joint</joint>
+        <joint>$(arg namespace)/wheel_right_joint</joint>
       </plugin>
     </gazebo>

Commit message: image bridge fixed, camera namespace added

File: kobuki_description/urdf/kobuki.urdf.xacro (robot description, xacro)
@@ -39,5 +39,5 @@
   <xacro:if value="$(arg camera)">
     <xacro:include filename="$(find kobuki_description)/urdf/sensors/asus_xtion_pro.urdf.xacro"/>
-    <xacro:sensor_asus_xtion_pro parent="$(arg namespace)/base_link"/>
+    <xacro:sensor_asus_xtion_pro parent="$(arg namespace)/base_link" namespace="$(arg namespace)"/>
   </xacro:if>
   <xacro:if value="$(arg gazebo)">

File: kobuki_description/urdf/kobuki_gazebo.urdf.xacro (robot description, xacro)
@@ -59,6 +59,6 @@
     </xacro:if>
     <xacro:if value="$(arg camera)">
-      <gazebo reference="camera_rgb_frame">
-        <sensor type="rgbd_camera" name="kobuki_frame_sensor">
+      <gazebo reference="$(arg namespace)/camera_rgb_frame">
+        <sensor type="rgbd_camera" name="$(arg namespace)/kobuki_frame_sensor">
           <always_on>1</always_on>
           <update_rate>30.0</update_rate>
@@ -83,5 +83,5 @@
               <p2>0.00000001</p2>
             </distortion>
-            <optical_frame_id>camera_rgb_optical_link</optical_frame_id>
+            <optical_frame_id>$(arg namespace)/camera_rgb_optical_link</optical_frame_id>
           </camera>
         </sensor>

File: kobuki_description/urdf/sensors/asus_xtion_pro.urdf.xacro (robot description, xacro)
@@ -8,25 +8,25 @@
   <xacro:property name="asus_xtion_pro_cam_rel_rgb_py"   value="-0.0220" />
   <!-- Parameterised in part by the values in turtlebot_properties.urdf.xacro -->
-  <xacro:macro name="sensor_asus_xtion_pro" params="parent">
-    <joint name="camera_rgb_joint" type="fixed">
+  <xacro:macro name="sensor_asus_xtion_pro" params="parent namespace">
+    <joint name="$(arg namespace)/camera_rgb_joint" type="fixed">
       <origin xyz="${cam_px} ${asus_xtion_pro_cam_py} ${cam_pz}"
               rpy="${cam_or} ${cam_op} ${cam_oy}"/>
       <parent link="${parent}"/>
-      <child link="camera_rgb_frame" />
+      <child link="$(arg namespace)/camera_rgb_frame" />
     </joint>
-    <link name="camera_rgb_frame"/>
+    <link name="$(arg namespace)/camera_rgb_frame"/>
     <joint name="camera_rgb_optical_joint" type="fixed">
       <origin xyz="0 0 0" rpy="0 0 0" />
-      <parent link="camera_rgb_frame" />
-      <child link="camera_rgb_optical_frame" />
+      <parent link="$(arg namespace)/camera_rgb_frame" />
+      <child link="$(arg namespace)/camera_rgb_optical_frame" />
     </joint>
-    <link name="camera_rgb_optical_frame"/>
-    <joint name="camera_joint" type="fixed">
+    <link name="$(arg namespace)/camera_rgb_optical_frame"/>
+    <joint name="$(arg namespace)/camera_joint" type="fixed">
       <origin xyz="0 ${asus_xtion_pro_cam_rel_rgb_py} 0"
               rpy="0 0 0"/>
-      <parent link="camera_rgb_frame"/>
-      <child link="camera_link"/>
+      <parent link="$(arg namespace)/camera_rgb_frame"/>
+      <child link="$(arg namespace)/camera_link"/>
     </joint>
-    <link name="camera_link">
+    <link name="$(arg namespace)/camera_link">
       <visual>
         <origin xyz="-0.015 0.0035 0.004" rpy="0 0 0"/>
@@ -49,16 +49,16 @@
       </inertial>
     </link>
-    <joint name="camera_depth_joint" type="fixed">
+    <joint name="$(arg namespace)/camera_depth_joint" type="fixed">
       <origin xyz="0 ${asus_xtion_pro_depth_rel_rgb_py} 0" rpy="0 0 0" />
-      <parent link="camera_rgb_frame" />
-      <child link="camera_depth_frame" />
+      <parent link="$(arg namespace)/camera_rgb_frame" />
+      <child link="$(arg namespace)/camera_depth_frame" />
     </joint>
-    <link name="camera_depth_frame"/>
-    <joint name="camera_depth_optical_joint" type="fixed">
+    <link name="$(arg namespace)/camera_depth_frame"/>
+    <joint name="$(arg namespace)/camera_depth_optical_joint" type="fixed">
       <origin xyz="0 0 0" rpy="0 0 0" />
-      <parent link="camera_depth_frame" />
-      <child link="camera_depth_optical_frame" />
+      <parent link="$(arg namespace)/camera_depth_frame" />
+      <child link="$(arg namespace)/camera_depth_optical_frame" />
     </joint>
-    <link name="camera_depth_optical_frame"/>
+    <link name="$(arg namespace)/camera_depth_optical_frame"/>
   </xacro:macro>
 </robot>

Commit message: added laser range as an argument for more flexibility

File: kobuki_description/urdf/kobuki.urdf.xacro (robot description, xacro)
@@ -9,4 +9,5 @@
   <xacro:arg name="camera" default="false" />
   <xacro:arg name="structure" default="false" />
+  <xacro:arg name="lidar_range" default="3.0" />
   <!-- Namespace will be applied to all TF frames and topics.
        This is required if multiple robots are launched at the same time.
@@ -54,5 +55,5 @@
   <xacro:if value="$(arg gazebo)">
     <xacro:include filename="$(find kobuki_description)/urdf/kobuki_gazebo.urdf.xacro"/>
-    <xacro:kobuki_gazebo lidar="$(arg lidar)" camera="$(arg camera)" namespace="$(arg namespace)" tf_namespace="$(arg tf_namespace)"/>
+    <xacro:kobuki_gazebo lidar="$(arg lidar)" camera="$(arg camera)" namespace="$(arg namespace)" tf_namespace="$(arg tf_namespace)" lidar_range="$(arg lidar_range)"/>
   </xacro:if>
 </robot>

File: kobuki_description/urdf/kobuki_gazebo.urdf.xacro (robot description, xacro)
@@ -1,5 +1,5 @@
 <?xml version="1.0" ?>
 <robot name="kobuki_gazebo" xmlns:xacro="http://ros.org/wiki/xacro">
-  <xacro:macro name="kobuki_gazebo" params="lidar camera namespace tf_namespace">
+  <xacro:macro name="kobuki_gazebo" params="lidar camera namespace tf_namespace lidar_range:=3.0">
     <gazebo>
       <plugin filename="gz-sim-diff-drive-system" name="gz::sim::systems::DiffDrive">
@@ -46,5 +46,5 @@
               <range>
                 <min>0.17</min>
-                <max>3.5</max>
+                <max>$(arg lidar_range)</max>
                 <resolution>0.015000</resolution>
               </range>
