Commit message: Reduced mass of the hexagons
Signed-off-by: Juancams <jc.manzanares.serrano@gmail.com>

File: kobuki_description/urdf/stacks/hexagons.urdf.xacro (robot description, xacro)
@@ -152,5 +152,5 @@
       </collision>
       <inertial>
-        <mass value="0.520" />
+        <mass value="0.100" />
         <origin xyz="0 0 0" />
         <inertia ixx="0.003328" ixy="0.0" ixz="0.0"
@@ -182,5 +182,5 @@
       </collision>
       <inertial>
-        <mass value="0.520" />
+        <mass value="0.100" />
         <origin xyz="0 0 0" />
         <inertia ixx="0.003328" ixy="0.0" ixz="0.0"
@@ -214,5 +214,5 @@
       </collision>
       <inertial>
-        <mass value="0.520"/>
+        <mass value="0.100"/>
         <origin xyz="0 0 0"/>
         <inertia ixx="0.003328" ixy="0.0" ixz="0.0"
