Commit message: updated all sensors and stacks with namespace and added namespace to bridge node

File: kobuki_description/urdf/sensors/astra.urdf.xacro (robot description, xacro)
@@ -9,25 +9,25 @@
   <xacro:property name="astra_dae_display_scale"   value="1" />
   <!-- Parameterised in part by the values in turtlebot_properties.urdf.xacro -->
-  <xacro:macro name="sensor_astra" params="parent">
-    <joint name="camera_rgb_joint" type="fixed">
+  <xacro:macro name="sensor_astra" params="parent namespace">
+    <joint name="$(arg namespace)/camera_rgb_joint" type="fixed">
       <origin xyz="${cam_px} ${astra_cam_py} ${cam_pz}"
               rpy="0 0 0"/>
       <parent link="${parent}"/>
-      <child link="camera_rgb_frame" />
+      <child link="$(arg namespace)/camera_rgb_frame" />
     </joint>
-    <link name="camera_rgb_frame"/>
-    <joint name="camera_rgb_optical_joint" type="fixed">
+    <link name="$(arg namespace)/camera_rgb_frame"/>
+    <joint name="$(arg namespace)/camera_rgb_optical_joint" type="fixed">
       <origin xyz="0 0 0" rpy="${-M_PI/2} 0 ${-M_PI/2}" />
-      <parent link="camera_rgb_frame" />
-      <child link="camera_rgb_optical_frame" />
+      <parent link="$(arg namespace)/camera_rgb_frame" />
+      <child link="$(arg namespace)/camera_rgb_optical_frame" />
     </joint>
-    <link name="camera_rgb_optical_frame"/>
-    <joint name="camera_joint" type="fixed">
+    <link name="$(arg namespace)/camera_rgb_optical_frame"/>
+    <joint name="$(arg namespace)/camera_joint" type="fixed">
       <origin xyz="0 ${astra_cam_rel_rgb_py} 0"
               rpy="0 0 0"/>
-      <parent link="camera_rgb_frame"/>
-      <child link="camera_link"/>
+      <parent link="$(arg namespace)/camera_rgb_frame"/>
+      <child link="$(arg namespace)/camera_link"/>
     </joint>
-    <link name="camera_link">
+    <link name="$(arg namespace)/camera_link">
       <visual>
         <origin xyz="-0.04 0.02 -0.01" rpy="${M_PI/2} 0 ${M_PI/2}"/>
@@ -50,16 +50,16 @@
       </inertial>
     </link>
-    <joint name="camera_depth_joint" type="fixed">
+    <joint name="$(arg namespace)/camera_depth_joint" type="fixed">
       <origin xyz="0 ${astra_depth_rel_rgb_py} 0" rpy="0 0 0" />
-      <parent link="camera_rgb_frame" />
-      <child link="camera_depth_frame" />
+      <parent link="$(arg namespace)/camera_rgb_frame" />
+      <child link="$(arg namespace)/camera_depth_frame" />
     </joint>
-    <link name="camera_depth_frame"/>
-    <joint name="camera_depth_optical_joint" type="fixed">
+    <link name="$(arg namespace)/camera_depth_frame"/>
+    <joint name="$(arg namespace)/camera_depth_optical_joint" type="fixed">
       <origin xyz="0 0 0" rpy="${-M_PI/2} 0 ${-M_PI/2}" />
-      <parent link="camera_depth_frame" />
-      <child link="camera_depth_optical_frame" />
+      <parent link="$(arg namespace)/camera_depth_frame" />
+      <child link="$(arg namespace)/camera_depth_optical_frame" />
     </joint>
-    <link name="camera_depth_optical_frame"/>
+    <link name="$(arg namespace)/camera_depth_optical_frame"/>
     <!-- RGBD sensor for simulation, same as Kinect -->
     <turtlebot_sim_3dsensor/>

File: kobuki_description/urdf/sensors/asus_xtion_pro.urdf.xacro (robot description, xacro)
@@ -16,5 +16,5 @@
     </joint>
     <link name="$(arg namespace)/camera_rgb_frame"/>
-    <joint name="camera_rgb_optical_joint" type="fixed">
+    <joint name="$(arg namespace)/camera_rgb_optical_joint" type="fixed">
       <origin xyz="0 0 0" rpy="0 0 0" />
       <parent link="$(arg namespace)/camera_rgb_frame" />

File: kobuki_description/urdf/sensors/asus_xtion_pro_offset.urdf.xacro (robot description, xacro)
@@ -9,25 +9,25 @@
   <xacro:property name="asus_xtion_pro_offset_cam_rel_rgb_py"   value="-0.0220" />
   <!-- Parameterised in part by the values in turtlebot_properties.urdf.xacro -->
-  <xacro:macro name="sensor_asus_xtion_pro_offset" params="parent">
+  <xacro:macro name="sensor_asus_xtion_pro_offset" params="parent namespace">
     <joint name="camera_rgb_joint" type="fixed">
       <origin xyz="${cam_px} ${asus_xtion_pro_offset_cam_py} ${cam_pz}"
               rpy="${cam_or} ${cam_op} ${cam_oy}"/>
       <parent link="${parent}"/>
-      <child link="camera_rgb_frame" />
+      <child link="$(arg namespace)/camera_rgb_frame" />
     </joint>
-    <link name="camera_rgb_frame"/>
-    <joint name="camera_rgb_optical_joint" type="fixed">
+    <link name="$(arg namespace)/camera_rgb_frame"/>
+    <joint name="$(arg namespace)/camera_rgb_optical_joint" type="fixed">
       <origin xyz="0 0 0" rpy="${-M_PI/2} 0 ${-M_PI/2}" />
-      <parent link="camera_rgb_frame" />
-      <child link="camera_rgb_optical_frame" />
+      <parent link="$(arg namespace)/camera_rgb_frame" />
+      <child link="$(arg namespace)/camera_rgb_optical_frame" />
     </joint>
-    <link name="camera_rgb_optical_frame"/>
-    <joint name="camera_joint" type="fixed">
+    <link name="$(arg namespace)/camera_rgb_optical_frame"/>
+    <joint name="$(arg namespace)/camera_joint" type="fixed">
       <origin xyz="0 ${asus_xtion_pro_offset_cam_rel_rgb_py} 0"
               rpy="0 0 0"/>
-      <parent link="camera_rgb_frame"/>
-      <child link="camera_link"/>
+      <parent link="$(arg namespace)/camera_rgb_frame"/>
+      <child link="$(arg namespace)/camera_link"/>
     </joint>
-    <link name="camera_link">
+    <link name="$(arg namespace)/camera_link">
       <visual>
         <origin xyz="-0.01 0 0" rpy="${-M_PI/2} -${M_PI} ${-M_PI/2}"/>
@@ -50,16 +50,16 @@
       </inertial>
     </link>
-    <joint name="camera_depth_joint" type="fixed">
+    <joint name="$(arg namespace)/camera_depth_joint" type="fixed">
       <origin xyz="0 ${asus_xtion_pro_offset_depth_rel_rgb_py} 0" rpy="0 0 0" />
-      <parent link="camera_rgb_frame" />
-      <child link="camera_depth_frame" />
+      <parent link="$(arg namespace)/camera_rgb_frame" />
+      <child link="$(arg namespace)/camera_depth_frame" />
     </joint>
-    <link name="camera_depth_frame"/>
-    <joint name="camera_depth_optical_joint" type="fixed">
+    <link name="$(arg namespace)/camera_depth_frame"/>
+    <joint name="$(arg namespace)/camera_depth_optical_joint" type="fixed">
       <origin xyz="0 0 0" rpy="${-M_PI/2} 0 ${-M_PI/2}" />
-      <parent link="camera_depth_frame" />
-      <child link="camera_depth_optical_frame" />
+      <parent link="$(arg namespace)/camera_depth_frame" />
+      <child link="$(arg namespace)/camera_depth_optical_frame" />
     </joint>
-    <link name="camera_depth_optical_frame"/>
+    <link name="$(arg namespace)/camera_depth_optical_frame"/>
     <!-- RGBD sensor for simulation, same as Kinect -->
     <turtlebot_sim_3dsensor/>

File: kobuki_description/urdf/sensors/kinect.urdf.xacro (robot description, xacro)
@@ -5,23 +5,23 @@
   <xacro:property name="kinect_cam_py" value="-0.0125"/>
   <!-- Parameterised in part by the values in turtlebot_properties.urdf.xacro -->
-  <xacro:macro name="sensor_kinect" params="parent">
-    <joint name="camera_rgb_joint" type="fixed">
+  <xacro:macro name="sensor_kinect" params="parent namespace">
+    <joint name="c$(arg namespace)/amera_rgb_joint" type="fixed">
       <origin xyz="${cam_px} ${kinect_cam_py} ${cam_pz}" rpy="${cam_or} ${cam_op} ${cam_oy}"/>
       <parent link="${parent}"/>
-      <child link="camera_rgb_frame" />
+      <child link="$(arg namespace)/camera_rgb_frame" />
     </joint>
-    <link name="camera_rgb_frame"/>
-    <joint name="camera_rgb_optical_joint" type="fixed">
+    <link name="$(arg namespace)/camera_rgb_frame"/>
+    <joint name="$(arg namespace)/camera_rgb_optical_joint" type="fixed">
       <origin xyz="0 0 0" rpy="${-M_PI/2} 0 ${-M_PI/2}" />
-      <parent link="camera_rgb_frame" />
-      <child link="camera_rgb_optical_frame" />
+      <parent link="$(arg namespace)/camera_rgb_frame" />
+      <child link="$(arg namespace)/camera_rgb_optical_frame" />
     </joint>
-    <link name="camera_rgb_optical_frame"/>
-    <joint name="camera_joint" type="fixed">
+    <link name="$(arg namespace)/camera_rgb_optical_frame"/>
+    <joint name="$(arg namespace)/camera_joint" type="fixed">
       <origin xyz="-0.031 ${-kinect_cam_py} -0.016" rpy="0 0 0"/>
-      <parent link="camera_rgb_frame"/>
-      <child link="camera_link"/>
+      <parent link="$(arg namespace)/camera_rgb_frame"/>
+      <child link="$(arg namespace)/camera_link"/>
     </joint>
-      <link name="camera_link">
+      <link name="$(arg namespace)/camera_link">
       <visual>
        <origin xyz="0 0 0" rpy="0 0 ${M_PI/2}"/>
@@ -47,16 +47,16 @@
          files. However, for Gazebo simulation we need them, so we add them here.
          (Hence, don't publish them additionally!) -->
-	<joint name="camera_depth_joint" type="fixed">
+	<joint name="$(arg namespace)/camera_depth_joint" type="fixed">
 	  <origin xyz="0 ${2 * -kinect_cam_py} 0" rpy="0 0 0" />
-	  <parent link="camera_rgb_frame" />
-	  <child link="camera_depth_frame" />
+	  <parent link="$(arg namespace)/camera_rgb_frame" />
+	  <child link="$(arg namespace)/camera_depth_frame" />
 	</joint>
-	<link name="camera_depth_frame"/>
-	<joint name="camera_depth_optical_joint" type="fixed">
+	<link name="$(arg namespace)/camera_depth_frame"/>
+	<joint name="$(arg namespace)/camera_depth_optical_joint" type="fixed">
 	  <origin xyz="0 0 0" rpy="${-M_PI/2} 0 ${-M_PI/2}" />
-	  <parent link="camera_depth_frame" />
-	  <child link="camera_depth_optical_frame" />
+	  <parent link="$(arg namespace)/camera_depth_frame" />
+	  <child link="$(arg namespace)/camera_depth_optical_frame" />
 	</joint>
-	<link name="camera_depth_optical_frame"/>
+	<link name="$(arg namespace)/camera_depth_optical_frame"/>
 	<!-- Kinect sensor for simulation -->
 	<turtlebot_sim_3dsensor/>

File: kobuki_description/urdf/sensors/r200.urdf.xacro (robot description, xacro)
@@ -21,15 +21,15 @@
   <xacro:property name="r200_cam_rgb_pz" value="0.013"/>
   <xacro:property name="r200_cam_depth_offset" value="0.01"/>
-  <xacro:macro name="sensor_r200" params="parent">
+  <xacro:macro name="sensor_r200" params="parent namespace">
     <!--
     ==  Mount and camera body joints & links ==
     -->
     <!-- right bracket end -->
-    <joint name="bracket_end_right_joint" type="fixed">
+    <joint name="$(arg namespace)/bracket_end_right_joint" type="fixed">
       <origin xyz="${pole_px} ${pole_py} ${pole_pz}" rpy="0 0 0"/>
       <parent link="${parent}"/>
-      <child link="bracket_end_right" />
+      <child link="$(arg namespace)/bracket_end_right" />
     </joint>
-    <link name="bracket_end_right">
+    <link name="$(arg namespace)/bracket_end_right">
     <visual>
        <origin xyz="${-r200_bracket_end_width/2} ${r200_bracket_end_offset_py} ${r200_bracket_end_offset_pz}" rpy="0 0 ${-M_PI/2}"/>
@@ -41,10 +41,10 @@
     </link>
     <!-- center main bracket -->
-    <joint name="bracket_joint" type="fixed">
+    <joint name="$(arg namespace)/bracket_joint" type="fixed">
       <origin xyz="${r200_bracket_width/2} ${r200_bracket_offset_py} ${r200_bracket_offset_pz}" rpy="0 0 0"/>
-      <parent link="bracket_end_right"/>
-      <child link="bracket" />
+      <parent link="$(arg namespace)/bracket_end_right"/>
+      <child link="$(arg namespace)/bracket" />
     </joint>
-    <link name="bracket">
+    <link name="$(arg namespace)/bracket">
     <visual>
        <origin xyz="0 0 0" rpy="0 0 ${M_PI/2}"/>
@@ -56,10 +56,10 @@
     </link>
     <!-- left bracket end -->
-    <joint name="bracket_end_left_joint" type="fixed">
+    <joint name="$(arg namespace)/bracket_end_left_joint" type="fixed">
       <origin xyz="${-r200_bracket_width/2} ${r200_bracket_length - r200_bracket_offset_py} ${-r200_bracket_offset_pz}" rpy="0 0 0"/>
-      <parent link="bracket"/>
-      <child link="bracket_end_left" />
+      <parent link="$(arg namespace)/bracket"/>
+      <child link="$(arg namespace)/bracket_end_left" />
     </joint>
-    <link name="bracket_end_left">
+    <link name="$(arg namespace)/bracket_end_left">
     <visual>
        <origin xyz="${r200_bracket_end_width/2} 0 ${-r200_bracket_end_offset_pz}" rpy="0 0 ${M_PI/2}"/>
@@ -71,10 +71,10 @@
     </link>
     <!-- camera body -->
-    <joint name="camera_joint" type="fixed">
+    <joint name="$(arg namespace)/camera_joint" type="fixed">
       <origin xyz="${r200_cam_offset_px} ${r200_cam_offset_py} ${r200_cam_offset_pz}" rpy="0 0 0"/>
-      <parent link="bracket"/>
-      <child link="camera_link" />
+      <parent link="$(arg namespace)/bracket"/>
+      <child link="$(arg namespace)/camera_link" />
     </joint>
-    <link name="camera_link">
+    <link name="$(arg namespace)/camera_link">
       <visual>
        <origin xyz="0 0 0" rpy="${M_PI/2} 0 ${M_PI/2}"/>
@@ -101,31 +101,31 @@
     ==  RGB joints & links ==
     -->
-    <joint name="camera_rgb_joint" type="fixed">
+    <joint name="$(arg namespace)/camera_rgb_joint" type="fixed">
       <origin xyz="${r200_cam_rgb_px} ${r200_cam_rgb_py} ${r200_cam_rgb_pz}" rpy="0 0 0"/>
-      <parent link="camera_link"/>
-      <child link="camera_rgb_frame" />
+      <parent link="$(arg namespace)/camera_link"/>
+      <child link="$(arg namespace)/camera_rgb_frame" />
     </joint>
-    <link name="camera_rgb_frame"/>
-    <joint name="camera_rgb_optical_joint" type="fixed">
+    <link name="$(arg namespace)/camera_rgb_frame"/>
+    <joint name="$(arg namespace)/camera_rgb_optical_joint" type="fixed">
       <origin xyz="0 0 0" rpy="${-M_PI/2} 0 ${-M_PI/2}" />
-      <parent link="camera_rgb_frame" />
-      <child link="camera_rgb_optical_frame" />
+      <parent link="$(arg namespace)/camera_rgb_frame" />
+      <child link="$(arg namespace)/camera_rgb_optical_frame" />
     </joint>
-    <link name="camera_rgb_optical_frame"/>
+    <link name="$(arg namespace)/camera_rgb_optical_frame"/>
     <!--
     ==  Depth joints & links ==
     -->
-    <joint name="camera_depth_joint" type="fixed">
+    <joint name="$(arg namespace)/camera_depth_joint" type="fixed">
         <origin xyz="0 ${r200_cam_depth_offset} 0" rpy="0 0 0" />
-        <parent link="camera_rgb_frame" />
-        <child link="camera_depth_frame" />
+        <parent link="$(arg namespace)/camera_rgb_frame" />
+        <child link="$(arg namespace)/camera_depth_frame" />
     </joint>
-    <link name="camera_depth_frame"/>
-    <joint name="camera_depth_optical_joint" type="fixed">
+    <link name="$(arg namespace)/camera_depth_frame"/>
+    <joint name="$(arg namespace)/camera_depth_optical_joint" type="fixed">
         <origin xyz="0 0 0" rpy="${-M_PI/2} 0 ${-M_PI/2}" />
-        <parent link="camera_depth_frame" />
-        <child link="camera_depth_optical_frame" />
+        <parent link="$(arg namespace)/camera_depth_frame" />
+        <child link="$(arg namespace)/camera_depth_optical_frame" />
     </joint>
-    <link name="camera_depth_optical_frame"/>
+    <link name="$(arg namespace)/camera_depth_optical_frame"/>
   	<!-- Simulation sensor -->
     <turtlebot_sim_3dsensor/>

File: kobuki_description/urdf/stacks/circles.urdf.xacro (robot description, xacro)
@@ -2,10 +2,10 @@
 <robot name="turtlebot_hardware" xmlns:xacro="http://ros.org/wiki/xacro">
   <xacro:macro name="turtlebot_spacer" params="parent number x_loc y_loc z_loc namespace">
-    <joint name="spacer_${number}_joint" type="fixed">
-      <origin xyz="${x_loc} ${y_loc} ${z_loc}" rpy="0 0 0" />
-      <parent link="${parent}"/>
-      <child link="spacer_${number}_link" />
-    </joint>
-    <link name="spacer_${number}_link">
+    <joint name="$(arg namespace)/spacer_${number}_joint" type="fixed">
+      <origin xyz="${x_loc} ${y_loc} ${z_loc}" rpy="0 0 0" />
+      <parent link="${parent}"/>
+      <child link="$(arg namespace)/spacer_${number}_link" />
+    </joint>
+    <link name="$(arg namespace)/spacer_${number}_link">
       <inertial>
         <mass value="0.001" />
@@ -114,10 +114,10 @@
   </xacro:macro>
   <xacro:macro name="turtlebot_standoff_kinect" params="parent number x_loc y_loc z_loc namespace">
-    <joint name="standoff_kinect_${number}_joint" type="fixed">
-      <origin xyz="${x_loc} ${y_loc} ${z_loc}" rpy="0 0 0" />
-      <parent link="${parent}"/>
-      <child link="standoff_kinect_${number}_link" />
-    </joint>
-    <link name="standoff_kinect_${number}_link">
+    <joint name="$(arg namespace)/standoff_kinect_${number}_joint" type="fixed">
+      <origin xyz="${x_loc} ${y_loc} ${z_loc}" rpy="0 0 0" />
+      <parent link="${parent}"/>
+      <child link="$(arg namespace)/standoff_kinect_${number}_link" />
+    </joint>
+    <link name="$(arg namespace)/standoff_kinect_${number}_link">
       <inertial>
         <mass value="0.001" />
@@ -146,10 +146,10 @@
     <turtlebot_spacer parent="${parent}" number="2" x_loc="-0.07239" y_loc="-0.1114679" z_loc="0.062992"/>
     <turtlebot_spacer parent="${parent}" number="3" x_loc="-0.07239" y_loc="0.1114679" z_loc="0.062992"/>
-    <joint name="plate_0_joint" type="fixed">
+    <joint name="$(arg namespace)/plate_0_joint" type="fixed">
       <origin xyz="-0.04334 0  0.06775704" rpy="0 0 0" />
       <parent link="${parent}"/>
-      <child link="plate_0_link" />
-    </joint>
-    <link name="plate_0_link">
+      <child link="$(arg namespace)/plate_0_link" />
+    </joint>
+    <link name="$(arg namespace)/plate_0_link">
       <inertial>
         <mass value="0.01" />
@@ -176,10 +176,10 @@
     <turtlebot_standoff_2in parent="${parent}" number="2" x_loc="-0.052832" y_loc="-0.1314196" z_loc="0.0709803"/>
     <turtlebot_standoff_2in parent="${parent}" number="3" x_loc="-0.052832" y_loc="0.1314196" z_loc="0.0709803"/>
-    <joint name="plate_1_joint" type="fixed">
+    <joint name="$(arg namespace)/plate_1_joint" type="fixed">
       <origin xyz="0.04068 0 0.05715" rpy="0 0 0" />
-      <parent link="plate_0_link"/>
-      <child link="plate_1_link" />
-    </joint>
-    <link name="plate_1_link">
+      <parent link="$(arg namespace)/plate_0_link"/>
+      <child link="$(arg namespace)/plate_1_link" />
+    </joint>
+    <link name="$(arg namespace)/plate_1_link">
       <inertial>
         <mass value="0.1" />
@@ -202,14 +202,14 @@
       </collision>
     </link>
-    <turtlebot_standoff_2in parent="standoff_2in_0_link" number="4" x_loc="0" y_loc="0" z_loc="0.05715"/>
-    <turtlebot_standoff_2in parent="standoff_2in_1_link" number="5" x_loc="0" y_loc="0" z_loc="0.05715"/>
-    <turtlebot_standoff_2in parent="standoff_2in_2_link" number="6" x_loc="0" y_loc="0" z_loc="0.05715"/>
-    <turtlebot_standoff_2in parent="standoff_2in_3_link" number="7" x_loc="0" y_loc="0" z_loc="0.05715"/>
-    <joint name="plate_2_joint" type="fixed">
+    <turtlebot_standoff_2in parent="$(arg namespace)standoff_2in_0_link" number="4" x_loc="0" y_loc="0" z_loc="0.05715"/>
+    <turtlebot_standoff_2in parent="$(arg namespace)standoff_2in_1_link" number="5" x_loc="0" y_loc="0" z_loc="0.05715"/>
+    <turtlebot_standoff_2in parent="$(arg namespace)standoff_2in_2_link" number="6" x_loc="0" y_loc="0" z_loc="0.05715"/>
+    <turtlebot_standoff_2in parent="$(arg namespace)standoff_2in_3_link" number="7" x_loc="0" y_loc="0" z_loc="0.05715"/>
+    <joint name="$(arg namespace)plate_2_joint" type="fixed">
       <origin xyz="0 0 0.0572008" rpy="0 0 0" />
       <parent link="plate_1_link"/>
       <child link="plate_2_link" />
     </joint>
-    <link name="plate_2_link">
+    <link name="$(arg namespace)plate_2_link">
       <inertial>
         <mass value="0.01" />
@@ -232,16 +232,16 @@
       </collision>
     </link>
-    <turtlebot_standoff_kinect parent="plate_2_link" number="0" x_loc="-0.1024382" y_loc="0.098" z_loc="0.0032004"/>
-    <turtlebot_standoff_kinect parent="plate_2_link" number="1" x_loc="-0.1024382" y_loc="-0.098" z_loc="0.0032004"/>
-    <turtlebot_standoff_8in parent="standoff_2in_4_link" number="0" x_loc="0" y_loc="0" z_loc="0.05715"/>
-    <turtlebot_standoff_8in parent="standoff_2in_5_link" number="1" x_loc="0" y_loc="0" z_loc="0.05715"/>
-    <turtlebot_standoff_8in parent="standoff_2in_6_link" number="2" x_loc="0" y_loc="0" z_loc="0.05715"/>
-    <turtlebot_standoff_8in parent="standoff_2in_7_link" number="3" x_loc="0" y_loc="0" z_loc="0.05715"/>
-    <joint name="plate_3_joint" type="fixed">
+    <turtlebot_standoff_kinect parent="$(arg namespace)plate_2_link" number="0" x_loc="-0.1024382" y_loc="0.098" z_loc="0.0032004"/>
+    <turtlebot_standoff_kinect parent="$(arg namespace)plate_2_link" number="1" x_loc="-0.1024382" y_loc="-0.098" z_loc="0.0032004"/>
+    <turtlebot_standoff_8in parent="$(arg namespace)standoff_2in_4_link" number="0" x_loc="0" y_loc="0" z_loc="0.05715"/>
+    <turtlebot_standoff_8in parent="$(arg namespace)standoff_2in_5_link" number="1" x_loc="0" y_loc="0" z_loc="0.05715"/>
+    <turtlebot_standoff_8in parent="$(arg namespace)standoff_2in_6_link" number="2" x_loc="0" y_loc="0" z_loc="0.05715"/>
+    <turtlebot_standoff_8in parent="$(arg namespace)standoff_2in_7_link" number="3" x_loc="0" y_loc="0" z_loc="0.05715"/>
+    <joint name="$(arg namespace)plate_3_joint" type="fixed">
       <origin xyz="-0.01316 0 0.2063496" rpy="0 0 0" />
-      <parent link="plate_2_link"/>
-      <child link="plate_3_link" />
-    </joint>
-    <link name="plate_3_link">
+      <parent link="$(arg namespace)plate_2_link"/>
+      <child link="$(arg namespace)plate_3_link" />
+    </joint>
+    <link name="$(arg namespace)plate_3_link">
       <inertial>
         <mass value="0.01" />
