Commit message: updated all sensors and stacks with namespace and added namespace to bridge node

File: kobuki_description/urdf/stacks/hexagons.urdf.xacro (robot description, xacro)
@@ -9,11 +9,11 @@
   <!-- Xacro macros -->
   <!-- Pole macros -->
-  <xacro:macro name="stack_bottom_pole" params="parent number x_loc y_loc z_loc ">
-    <joint name="pole_bottom_${number}_joint" type="fixed">
+  <xacro:macro name="stack_bottom_pole" params="parent number x_loc y_loc z_loc namespace">
+    <joint name="$(arg namespace)/pole_bottom_${number}_joint" type="fixed">
       <origin xyz="${x_loc} ${y_loc} ${z_loc}" rpy="0 0 0"/>
       <parent link="${parent}"/>
-      <child link="pole_bottom_${number}_link"/>
-    </joint>
-    <link name="pole_bottom_${number}_link">
+      <child link="$(arg namespace)/pole_bottom_${number}_link"/>
+    </joint>
+    <link name="$(arg namespace)/pole_bottom_${number}_link">
       <visual>
         <origin xyz="0 0 0" rpy="0 0 0"/>
@@ -37,11 +37,11 @@
     </link>
   </xacro:macro>
-  <xacro:macro name="stack_middle_pole" params="parent number x_loc y_loc z_loc ">
-    <joint name="pole_middle_${number}_joint" type="fixed">
+  <xacro:macro name="stack_middle_pole" params="parent number x_loc y_loc z_loc namespace">
+    <joint name="$(arg namespace)/pole_middle_${number}_joint" type="fixed">
       <origin xyz="${x_loc} ${y_loc} ${z_loc}" rpy="0 0 0" />
       <parent link="${parent}"/>
-      <child link="pole_middle_${number}_link"/>
-    </joint>
-    <link name="pole_middle_${number}_link">
+      <child link="$(arg namespace)/pole_middle_${number}_link"/>
+    </joint>
+    <link name="$(arg namespace)/pole_middle_${number}_link">
       <visual>
         <origin xyz="0 0 0" rpy="0 ${M_PI} 0"/>
@@ -65,11 +65,11 @@
     </link>
   </xacro:macro>
-  <xacro:macro name="stack_top_pole" params="parent number x_loc y_loc z_loc ">
-    <joint name="pole_top_${number}_joint" type="fixed">
+  <xacro:macro name="stack_top_pole" params="parent number x_loc y_loc z_loc namespace ">
+    <joint name="$(arg namespace)/pole_top_${number}_joint" type="fixed">
       <origin xyz="${x_loc} ${y_loc} ${z_loc}" rpy="0 0 0"/>
       <parent link="${parent}"/>
-      <child link="pole_top_${number}_link"/>
-    </joint>
-    <link name="pole_top_${number}_link">
+      <child link="$(arg namespace)/pole_top_${number}_link"/>
+    </joint>
+    <link name="$(arg namespace)/pole_top_${number}_link">
       <visual>
         <origin xyz=" 0 0 0" rpy="0 0 0"/>
@@ -93,11 +93,11 @@
     </link>
   </xacro:macro>
-  <xacro:macro name="stack_3d_sensor_pole" params="parent number x_loc y_loc z_loc ">
-    <joint name="pole_kinect_${number}_joint" type="fixed">
+  <xacro:macro name="stack_3d_sensor_pole" params="parent number x_loc y_loc z_loc namespace ">
+    <joint name="$(arg namespace)/pole_kinect_${number}_joint" type="fixed">
       <origin xyz="${x_loc} ${y_loc} ${z_loc}" rpy="0 0 0"/>
       <parent link="${parent}"/>
-      <child link="pole_kinect_${number}_link"/>
-    </joint>
-    <link name="pole_kinect_${number}_link">
+      <child link="$(arg namespace)/pole_kinect_${number}_link"/>
+    </joint>
+    <link name="$(arg namespace)/pole_kinect_${number}_link">
       <visual>
         <origin xyz="0 0 -0.01" rpy="0 0 0"/>
