Commit message: Fix camera joints
Signed-off-by: Juancams <jc.manzanares.serrano@gmail.com>

File: kobuki_description/urdf/sensors/asus_xtion_pro.urdf.xacro (robot description, xacro)
@@ -17,5 +17,5 @@
     <link name="$(arg namespace)camera_rgb_frame"/>
     <joint name="$(arg namespace)camera_rgb_optical_joint" type="fixed">
-      <origin xyz="0 0 0" rpy="0 0 0" />
+      <origin xyz="0 0 0" rpy="${-M_PI/2} 0 ${-M_PI/2}" />
       <parent link="$(arg namespace)camera_rgb_frame" />
       <child link="$(arg namespace)camera_rgb_optical_frame" />
@@ -56,5 +56,5 @@
     <link name="$(arg namespace)camera_depth_frame"/>
     <joint name="$(arg namespace)camera_depth_optical_joint" type="fixed">
-      <origin xyz="0 0 0" rpy="0 0 0" />
+      <origin xyz="0 0 0" rpy="${-M_PI/2} 0 ${-M_PI/2}" />
       <parent link="$(arg namespace)camera_depth_frame" />
       <child link="$(arg namespace)camera_depth_optical_frame" />
