Commit message: Error with position
Signed-off-by: Juancams <jc.manzanares.serrano@gmail.com>

File: kobuki_description/urdf/sensors/lidar.urdf.xacro (robot description, xacro)
@@ -18,5 +18,5 @@
       </link>
       <joint name="laser_joint" type="fixed">
-        <origin xyz="0.0 0.0 0.37" rpy="0 0 0" />
+        <origin xyz="0.0 0.0 0.37" rpy="0 0 3.14" />
         <parent link="base_link"/>
         <child link="laser_link" />

Commit message: new world warehouses added

File: kobuki_description/urdf/sensors/lidar.urdf.xacro (robot description, xacro)
@@ -18,5 +18,5 @@
       </link>
       <joint name="$(arg namespace)/laser_joint" type="fixed">
-        <origin xyz="0.0 0.0 0.37" rpy="0 0 0" />
+        <origin xyz="0.0 0.0 0.37" rpy="0 0 3.14" />
         <parent link="$(arg namespace)/base_link"/>
         <child link="$(arg namespace)/laser_link" />

Commit message: Update laser_joint orientation in lidar.urdf.xacro
Now lidar is ok

File: kobuki_description/urdf/sensors/lidar.urdf.xacro (robot description, xacro)
@@ -18,5 +18,5 @@
       </link>
       <joint name="$(arg namespace)laser_joint" type="fixed">
-        <origin xyz="0.0 0.0 0.37" rpy="0 0 3.14" />
+        <origin xyz="0.0 0.0 0.37" rpy="0 0 0" />
         <parent link="$(arg namespace)base_link"/>
         <child link="$(arg namespace)laser_link" />
